File: analog.sch (KiCad schematic (older format))
At the start: 20 parts, among them U8 MAX11125

Commit message: First pass cleanup
Parts:
- removed AUDIO1: JACK_TRS_6PINS, audio-jack:CUI_SJ-43516-SMT, symbol jack_trs_6pins_apple:JACK_TRS_6PINS_APPLE
- removed C58, C61: 22uF, Capacitor_SMD:C_0805_2012Metric, symbol Device:C
- removed C59, C62: 220nF, Capacitor_SMD:C_0603_1608Metric, symbol Device:C
- removed L4, L5: 33uH, Inductor_SMD:L_0805_2012Metric_Pad1.15x1.40mm_HandSolder, symbol Device:L_Small
- removed R14, R18, R57: 1.1k, Resistor_SMD:R_0603_1608Metric, symbol Device:R
- removed R15, R19, R58: 549, Resistor_SMD:R_0603_1608Metric, symbol Device:R
- removed R16, R20, R59: 270, Resistor_SMD:R_0603_1608Metric, symbol Device:R
- removed R17, R21, R60: 130, Resistor_SMD:R_0603_1608Metric, symbol Device:R
- removed U8: MAX11125, max1112x-tqfn28:MAX1112x-TQFN-28-1EP_5x5mm_Pitch0.5mm, symbol max1112x:MAX1112x
Connections:
- net labels removed: +3V3, ADC3V3, ADCD3V3, ADC_CSn, ADC_MISO, ADC_MOSI, ADC_SCLK, AUDIO_L, AUDIO_L0, AUDIO_L1, AUDIO_L2, AUDIO_L3, AUDIO_R, AUDIO_R0, AUDIO_R1, AUDIO_R2, AUDIO_R3, AUDIO_V, AUDIO_V0, AUDIO_V1, AUDIO_V2, AUDIO_V3, GN14, GN15, GN16, GN17, GND, GP14, GP15, GP16, GP17
- wire segments 59 -> 0
- no-connect marks 4 -> 0
Other:
- note removed: "ADC SPI connected to\nBANK3 of "ram" sheet"
- note removed: "Audio connected to\nBANK7 on "gpio" sheet"
- note removed: "JACK pinout for SJ-43516-SMT-TR\nhttp://www.cui.com/product/resource/sj-4351x-smt-series.pdf\npin 1 - sleeve (GND)\npin 2 - tip (left channel)\npin 3 - ring1 (right channel)\npin 4 - ring2 (video)\npin 5 - tip switch\npin 6 - ring1 switch"
- note removed: "Output resistance: 75 ohm\nInternal resistance of FPGA pin: 10 ohm\n1/(1/(130+10)+1/(270+10)+1/(549+10)+1/(1100+10))=74.6"
