File: gpio.sch (KiCad schematic (older format))
At the start: 5 parts, among them J1 CONN_02X20, J2 CONN_02X20, U1 LFE5U-85F-6BG381C

Commit message: First pass cleanup
Parts:
- removed D51, D52: 0, jumper:D_SMA_Jumper_NC, symbol Device:Jumper_NC_Small
- removed J1, J2: CONN_02X20, Socket_Strips:Socket_Strip_Angled_2x20, symbol Connector_Generic:Conn_02x20_Odd_Even
Connections:
- net labels removed: +3V3, +5V, 2V5_3V3, GN14, GN15, GN16, GN17, GN18, GN19, GN20, GN21, GN22, GN23, GN24, GN25, GN26, GN27, GND, GP14, GP15, GP16, GP17, GP18, GP19, GP20, GP21, GP22, GP23, GP24, GP25, GP26, GP27, IN5V, OUT5V
- wire segments 24 -> 0
Other:
- note removed: "0"
- note removed: "1"
- note removed: "10"
- note removed: "11"
- note removed: "12"
- note removed: "13"
- note removed: "14"
- note removed: "15"
- note removed: "16"
- note removed: "17"
- note removed: "18"
- note removed: "19"
- note removed: "2"
- note removed: "20"
- note removed: "21"
- note removed: "22"
- note removed: "23"
- note removed: "24"
- note removed: "25"
- note removed: "26"
- note removed: "27"
- note removed: "3"
- note removed: "4"
- note removed: "5"
- note removed: "6"
- note removed: "7"
- note removed: "8"
- note removed: "9"
- note removed: "DAC WIFI_GPIO25"
- note removed: "DAC WIFI_GPIO26"
- note removed: "GP,GN 0-7 single-ended connected to BANK0\nGP,GN 8-13 differential bidirectional connected to BANK7"
- note removed: "GP,GN 14-21 differential bidirectional connected to BANK2,3 on "ram" sheet\nGP,GN 22-27 single-ended connected to BANK1 on "gpdi" sheet"
- note removed: "GR_PCLK0_0"
- note removed: "GR_PCLK0_1"
- note removed: "GR_PCLK3_0"
- note removed: "GR_PCLK7_1"
- note removed: "J1 J2 PIN numbering 1-40 is for FEMALE 90° ANGLED header.\nFor MALE VERTICAL header, SWAP EVEN and ODD pin numbers."
- note removed: "PCLKC0_0"
- note removed: "PCLKC0_1"
- note removed: "PCLKC7_1"
- note removed: "PCLKT0_0"
- note removed: "PCLKT0_1"
- note removed: "PCLKT7_1"
- note removed: "STPS2L40AF"
