File: power.sch (KiCad schematic (older format))
At the start: 84 parts, among them J5 VJ1, Q1 BC857, Q2 2N7002, U1 LFE5U-85F-6BG381C, U3 TLV62569DBV, U4 TLV62569DBV, U5 TLV62569DBV, U7 MCP7940NT, Y2 32768Hz

Commit message: First pass cleanup
Parts:
- removed B0: PTS645, Button_Switch_SMD:SW_SPST_PTS645, symbol Switch:SW_Push
- removed BAT1: CR1225, Keystone_3000_1x12mm-CoinCell:Keystone_3000_1x12mm-CoinCell, symbol Device:Battery_Cell
- removed C14, C60: 220nF, Capacitor_SMD:C_0603_1608Metric, symbol Device:C
- removed C47: 2.2uF, Capacitor_SMD:C_0805_2012Metric, symbol Device:C
- removed C54, C55: 22uF, Capacitor_SMD:C_0805_2012Metric, symbol Device:C
- removed C56, C57: 4.7pF, Capacitor_SMD:C_0603_1608Metric, symbol Device:C
- removed D10, D13, D14, D16, D17, D27: 1N914, Diode_SMD:D_SOD-323_HandSoldering, symbol Device:D
- removed D11: RED, LED_SMD:LED_0805_2012Metric, symbol Device:LED_ALT
- removed D12, D15: BAT54W, Diode_SMD:D_SOD-323_HandSoldering, symbol Device:D_Schottky
- removed J5: VJ1, Connector_PinHeader_2.54mm:PinHeader_1x03_P2.54mm_Vertical, symbol Connector_Generic:Conn_01x03
- removed Q1: BC857, Package_TO_SOT_SMD:SOT-23, symbol Device:Q_PNP_BEC
- removed Q2: 2N7002, Package_TO_SOT_SMD:SOT-23, symbol Device:Q_NMOS_GSD
- removed R1, R3, R4: 4.7k, Resistor_SMD:R_0603_1608Metric, symbol Device:R
- removed R10: 130, Resistor_SMD:R_0603_1608Metric, symbol Device:R
- removed R13: 15k, Resistor_SMD:R_0603_1608Metric, symbol Device:R
- removed R2: 18k, Resistor_SMD:R_0603_1608Metric, symbol Device:R
- removed R5: 2.2M, Resistor_SMD:R_0603_1608Metric, symbol Device:R
- removed R6, R66, R8: 1.1k, Resistor_SMD:R_0603_1608Metric, symbol Device:R
- removed R65: 549, Resistor_SMD:R_0603_1608Metric, symbol Device:R
- removed RV2: 0, Resistor_SMD:R_0805_2012Metric_Pad1.29x1.40mm_HandSolder, symbol Device:Jumper_NO_Small
- removed RV3: 0, Resistor_SMD:R_0805_2012Metric_Pad1.29x1.40mm_HandSolder, symbol Device:Jumper_NC_Small
- removed U7: MCP7940NT, SOT96-1:SOT96-1, symbol Timer_RTC:PCF8563T
- removed Y2: 32768Hz, abs25:Crystal_SMD_ABS25, symbol Device:Crystal_GND23
- C13: Digike_y2 1276-2903-1-ND -> (none); Digikey 587-5918-1-ND -> (none); Koncar FC001 -> (none); LCSC C87995 -> (none); Mouse_r2 603-CC805MRX5R6BB225 -> (none); Mouser 80-C0805C225K4R3123 -> (none)
Connections:
- net labels removed: BTN_PWRn, FPDI_SCL, FPDI_SDA, FTDI_nSLEEP, FTDI_nSUSPEND, HOLD, OSCI_32k, OSCO_32k, PWRBTn, RTCVDD, SHD, SHUT, SHUTDOWN, US2_ID, VBAT, WAKE, WAKEUPn, WKUP, WKn
- wire segments 450 -> 368
- no-connect marks 2 -> 0
Other:
- note removed: "D11 (2V), R2, R4 hold PWREN on 1V\nin the middle of 0.4-1.5V hysteresis"
- note removed: "D13 discharges\nC13 at shutdown"
- note removed: "D14 discharges\nC14 at shutdown"
- note removed: "FTDI_nSLEEP is 2.5V\nD12 must be schottky"
- note removed: "R5, C14 to hold 0.5s shutdown"
- note removed: "RC network for proper switchover\nto battery at fast fall of VDD.\nSee page 54 NXP PCF8523T datasheet.\nRTC can also be powered from 2.5V\nbut it is easier to route 3.3V"
- note removed: "SHUTDOWN connected to\nBANK2 on "ram" sheet"
- note removed: "WAKEUPn\nopen drain \nactive low"
- note removed: "WARNING\nECP5 family datasheet\np.48: Power Supply Ramp rates\nfor all supplies 0.01-10V/ms\n"
- note removed: "Works without R5"
- note removed: "to PROGRAMN\non "flash" sheet"
