File: ram.sch (KiCad schematic (older format))
At the start: 7 parts, among them U1 LFE5U-85F-6BG381C, U9 MT48LC16M16A2TG

Commit message: First pass cleanup
Parts:
- removed C16: 2.2uF, Capacitor_SMD:C_0805_2012Metric, symbol Device:C
- removed C33, C34, C35, C52: 22nF, Capacitor_SMD:C_0603_1608Metric, symbol Device:C
- removed U9: MT48LC16M16A2TG, TSOP54:TSOP54, symbol mt48lc16m16a2tg:MT48LC16M16A2TG
Connections:
- net labels removed: +3V3, GND
- wire segments 28 -> 0
