File: wifi.sch (KiCad schematic (older format))
At the start: 8 parts, among them J3 WIFI_OFF, U9 ESP32

Commit message: First pass cleanup
Parts:
- removed C15, C21: 22uF, Capacitor_SMD:C_0805_2012Metric, symbol Device:C
- removed J3: WIFI_OFF, Connector_PinHeader_2.54mm:PinHeader_1x02_P2.54mm_Vertical, symbol Connector_Generic:Conn_02x01
- removed R34: 15k, Resistor_SMD:R_0603_1608Metric, symbol Device:R
- removed R35: 549, Resistor_SMD:R_0603_1608Metric, symbol Device:R
- removed R38: 0.47, Resistor_SMD:R_0603_1608Metric, symbol Device:R
- removed SD1: 104031-0811, micro-sd-104031-811:MOLEX_104031-0811, symbol micro_sd_slide:104031-0811
- removed U9: ESP32, ESP32:ESP32, symbol esp32:ESP32-WROOM-WROVER
Connections:
- net labels removed: +3V3, GN12, GN13, GND, GP12, GP13, JTAG_TCK, JTAG_TDI, JTAG_TDO, JTAG_TMS, SD3V3, SD_CLK, SD_CMD, SD_D0, SD_D1, SD_D2, SD_D3, WIFIEN, WIFI_EN, WIFI_GPIO0, WIFI_GPIO19, WIFI_GPIO21, WIFI_GPIO22, WIFI_GPIO25, WIFI_GPIO26, WIFI_GPIO27, WIFI_GPIO35, WIFI_RXD, WIFI_TXD
- wire segments 23 -> 0
- no-connect marks 4 -> 0
Other:
- note removed: "ESP32 ADC capable pins\nGPIO36,39,34,35,32,33,25,26,27,\nGPIO14,12,13,15 - shared with HSPI/JTAG\nConnected to BANK7 on "gpio" sheet"
- note removed: "ESP32 HSPI pins\nGPIO12: MISO\nGPIO13: MOSI\nGPIO14: SCK\nGPIO15: SS"
- note removed: "ESP32 JTAG slave interface\nEN: TRST_N\nGPIO15: TDO\nGPIO12: TDI\nGPIO13: TCK\nGPIO14: TMS\nFLASH over JTAG\nnot yet supported."
- note removed: "ESP32 VSPI pins\nGPIO5: SS\nGPIO18: SCK\nGPIO19: MISO\nGPIO23: MOSI"
- note removed: "GN10 v1.7"
- note removed: "GN11 <v3.1 GP11 <v2.0.6"
- note removed: "GN12 <v3.1 GP12 <v2.0.6"
- note removed: "GN13 <v3.1"
- note removed: "GN9 v1.7"
- note removed: "GP11 <v3.1 GN11 <v2.0.6"
- note removed: "GP12 <v3.1 GN12 <v2.0.6"
- note removed: "GP13 <v2.0.6"
- note removed: "GP13 <v3.1 GN13 <v2.0.6"
- note removed: "GP9 v1.7"
- note removed: "GPIO12 probably should be held low at reset or disconnected\nother option is to burn flash voltage efuse for 3.3V operation\nfor GPIO2 and GPIO12 bootstrapping considerations, read\nhttps://github.com/espressif/esp-idf/tree/master/examples/storage/sd_card"
- note removed: "GPIO25,26 are DAC channels that can directly replay\naudio material over i2s bus"
- note removed: "NC <v3.1 GP10 v1.7 GP10 <=v3.1.2"
- note removed: "NC >=v3.1.2"
- note removed: "NC v1.7"
- note removed: "NC v1.7, >=v3.1.2"
- note removed: "NC v1.7, WIFI_GPIO5 <v3.1"
- note removed: "Programming pins:\nTXD RXD EN GPIO0"
- note removed: "SD card connected according to\nArduino->Examples->ESP32->SD_MMC_Test\nhttps://github.com/espressif/esp-idf/blob/\nmaster/examples/storage/sd_card/README.md\n"
- note removed: "SDcard connected to\nBANK6 on "usb" sheet"
- note removed: "Strapping pins\n(avoid using to avoid\nboot problems)\nGPIO0,2,4,5,12,15"
- note removed: "TDO <v3.1"
- note removed: "WIFI_GPIO15 v1.7"
- note removed: "WIFI_LED v1.7"
- note removed: "WROVER GPIO16,17\nused internally for PSRAM"
- note removed: "WiFi and SDcard connected to\nBANK6 on "usb" sheet"
- note removed: "minimum pins for compatible mode\nSD_CLK, SD_CMD, SD_D0, SD_D3"
