File: blinkey.sch (KiCad schematic (older format))
At the start: 34 parts, among them SW1 SW_DIP_x04

Commit message: First pass cleanup
Parts:
- removed B1, B2, B3, B4, B5, B6: PTS645, Button_Switch_SMD:SW_SPST_PTS645, symbol Switch:SW_Push
- removed D0, D4: RED, LED_SMD:LED_0805_2012Metric, symbol Device:LED_ALT
- removed D1, D5: ORANGE, LED_SMD:LED_0805_2012Metric, symbol Device:LED_ALT
- removed D2, D6: GREEN, LED_SMD:LED_0805_2012Metric, symbol Device:LED_ALT
- removed D3, D7: BLUE, LED_SMD:LED_0805_2012Metric, symbol Device:LED_ALT
- removed LCD1: ST7789, st7789:st7789, symbol st7789:ST7789
- removed R39, R51, R7: 130, Resistor_SMD:R_0603_1608Metric, symbol Device:R
- removed R41, R42, R43, R44, R45, R46, R47, R48: 549, Resistor_SMD:R_0603_1608Metric, symbol Device:R
- removed SW1: SW_DIP_x04, dipswitch:SW_DIP_x4_W8.61mm_Slide_LowProfile, symbol Switch:SW_DIP_x04
Connections:
- net labels removed: 2V5_3V3, ALED0, ALED1, ALED2, ALED3, ALED4, ALED5, ALED6, ALED7, BTNPUL, BTNPUR, BTN_D, BTN_F1, BTN_F2, BTN_L, BTN_R, BTN_U, LED0, LED1, LED2, LED3, LED4, LED5, LED6, LED7, OLED_BL, OLED_CLK, OLED_CS, OLED_DC, OLED_MOSI, OLED_RES, SW1, SW2, SW3, SW4, SWPU
- wire segments 67 -> 7
Other:
- note removed: "BTN_R,U to BANK2,3 on "ram" sheet\nBTN_F1,F2,D,L to BANK8 on "flash" sheet"
- note removed: "DIP switch connected to\nBANK0 on 'gpio' sheet"
- note removed: "DOWN"
- note removed: "FIRE1"
- note removed: "FIRE2"
- note removed: "LEDs connected to\nBANK7 on "gpio" sheet"
- note removed: "LEFT"
- note removed: "OLED connected to\nBANK6 on "usb" sheet"
- note removed: "RIGHT"
- note removed: "ST7789/SSD1331/SSD1351/SSD1306\ncompatible LCD/OLED 0.96/1.3/1.54" PCB \n14x14 units\n1 unit = 2.54 mm"
- note removed: "To fix issues with FT231XS rev A,B,C\nShort-circuit D18 LED, but then\nboard cannot keep awake by USB.\nchip rev D works properly\nSee TN140_FT231X Errata\n"
- note removed: "UP"

Commit message: More cleanup - moving flash and crystal
Parts:
- removed D18: GREEN, LED_SMD:LED_0805_2012Metric, symbol Device:LED
- removed D19: RED, LED_SMD:LED_0805_2012Metric, symbol Device:LED_ALT
- removed D22: BLUE, LED_SMD:LED_0805_2012Metric, symbol Device:LED
- removed R36, R37, R62: 549, Resistor_SMD:R_0603_1608Metric, symbol Device:R
Connections:
- net labels removed: FT2V5, FTDI_nSLEEP, FTDI_nTXLED, JTAG_TMS, LED_PWREN, LED_TXLED, LED_WIFI
- wire segments 7 -> 0
Other:
- note removed: "TXLED blinks when FPGA sends data to FTDI"
- note removed: "WIFI_GPIO2 v1.7, WIFI_GPIO5 <v3.1"
Changed lines of the file:
@@
 Comment4 ""
 $EndDescr
-Text GLabel 5650 4600 2    60   Input ~ 0
-FTDI_nSLEEP
-$Comp
-L Device:R R36
-U 1 1 590B507C
-P 4550 4600
-F 0 "R36" V 4630 4600 50  0000 C CNN
-F 1 "549" V 4550 4600 50  0000 C CNN
-F 2 "Resistor_SMD:R_0603_1608Metric" V 4480 4600 50  0001 C CNN
-F 3 "" H 4550 4600 50  0000 C CNN
-	1    4550 4600
-	0    1    1    0
-$EndComp
-Wire Wire Line
-	4700 4600 5350 4600
-Text Label 4750 4600 0    60   ~ 0
-LED_PWREN
-Wire Wire Line
-	4400 4600 4250 4600
-Wire Wire Line
-	4250 4600 4250 4950
-$Comp
-L power:GND #PWR084
-U 1 1 590B5B6D
-P 4250 4950
-F 0 "#PWR084" H 4250 4700 50  0001 C CNN
-F 1 "GND" H 4250 4800 50  0000 C CNN
-F 2 "" H 4250 4950 50  0000 C CNN
-F 3 "" H 4250 4950 50  0000 C CNN
-	1    4250 4950
-	1    0    0    -1
-$EndComp
-Text GLabel 5650 5350 2    60   Input ~ 0
-FTDI_nTXLED
-$Comp
-L Device:LED_ALT D19
-U 1 1 590B86F4
-P 4550 5350
-F 0 "D19" H 4550 5450 50  0000 C CNN
-F 1 "RED" H 4550 5250 50  0000 C CNN
-F 2 "LED_SMD:LED_0805_2012Metric" H 4550 5350 50  0001 C CNN
-F 3 "https://optoelectronics.liteon.com/upload/download/DS-22-99-0150/LTST-C170KRKT.pdf" H 4550 5350 50  0001 C CNN
-F 4 "www.liteon.com" H 4550 5350 60  0001 C CNN "MNF1_URL"
-F 5 "LTST-C170KRKT" H 4550 5350 60  0001 C CNN "MPN"
-F 6 "www.mouser.com" H 4550 5350 60  0001 C CNN "Mouser_URL"
-	1    4550 5350
-	-1   0    0    1
-$EndComp
-$Comp
-L Device:R R37
-U 1 1 590B86FA
-P 5500 5350
-F 0 "R37" V 5580 5350 50  0000 C CNN
-F 1 "549" V 5500 5350 50  0000 C CNN
-F 2 "Resistor_SMD:R_0603_1608Metric" V 5430 5350 50  0001 C CNN
-F 3 "" H 5500 5350 50  0000 C CNN
-	1    5500 5350
-	0    1    1    0
-$EndComp
-Wire Wire Line
-	4700 5350 5350 5350
-Text Label 4750 5350 0    60   ~ 0
-LED_TXLED
-Text GLabel 4300 5350 0    60   Input ~ 0
-FT2V5
-Wire Wire Line
-	4300 5350 4400 5350
-Text GLabel 5650 5850 2    60   Input ~ 0
-JTAG_TMS
-$Comp
-L Device:R R62
-U 1 1 5A07AFD8
-P 4550 5850
-F 0 "R62" V 4630 5850 50  0000 C CNN
-F 1 "549" V 4550 5850 50  0000 C CNN
-F 2 "Resistor_SMD:R_0603_1608Metric" V 4480 5850 50  0001 C CNN
-F 3 "" H 4550 5850 50  0000 C CNN
-	1    4550 5850
-	0    1    1    0
-$EndComp
-Wire Wire Line
-	4700 5850 5350 5850
-Text Label 4750 5850 0    60   ~ 0
-LED_WIFI
-Wire Wire Line
-	4400 5850 4250 5850
-Text Notes 6350 5400 0    60   ~ 0
-TXLED blinks when FPGA sends data to FTDI
-Text Notes 6400 5900 0    60   ~ 0
-WIFI_GPIO2 v1.7, WIFI_GPIO5 <v3.1
 $Comp
 L Device:C C46
@@
 	1    0    0    -1
 $EndComp
-$Comp
-L Device:LED D22
-U 1 1 5B988C80
-P 5500 5850
-F 0 "D22" H 5500 5950 50  0000 C CNN
-F 1 "BLUE" H 5600 5750 50  0000 R CNN
-F 2 "LED_SMD:LED_0805_2012Metric" H 5500 5850 50  0001 C CNN
-F 3 "http://optoelectronics.liteon.com/upload/download/DS-22-99-0226/LTST-C170TBKT.pdf" H 5500 5850 50  0001 C CNN
-F 4 "www.liteon.com" H 5500 5850 60  0001 C CNN "MNF1_URL"
-F 5 "LTST-C170TBKT" H 5500 5850 60  0001 C CNN "MPN"
-F 6 "http://optoelectronics.liteon.com/upload/download/ds22-2000-233/ltst-c171tbkt(0630).pdf" H 5500 5850 50  0001 C CNN "Datasheet2"
-F 7 "LTST-C171TBKT" H 5500 5850 50  0001 C CNN "MP_N2"
-F 8 "https://www.rohm.com/datasheet/SML-M13UT" H 5500 5850 50  0001 C CNN "Datasheet3"
-F 9 "SMLMN2BCTT86C" H 5500 5850 50  0001 C CNN "MP_N3"
-F 10 "859-LTST-C170TBKT" H 5500 5850 60  0001 C CNN "Mouser"
-F 11 "593-LSM0805463V" H 5500 5850 50  0001 C CNN "Mouse_r1"
-F 12 "755-SMLMN2BCTT86C" H 5500 5850 50  0001 C CNN "Mouse_r2"
-F 13 "859-LTST-C171TBKT" H 5500 5850 50  0001 C CNN "Mouse_r3"
-F 14 "160-1579-1-ND" H 5500 5850 50  0001 C CNN "Digikey"
-F 15 "C375453" H 5500 5850 50  0001 C CNN "LCSC"
-F 16 "FV004" H 5500 5850 50  0001 C CNN "Koncar"
-F 17 "T" H 5500 5850 50  0001 C CNN "Side"
-	1    5500 5850
-	-1   0    0    1
-$EndComp
-$Comp
-L Device:LED D18
-U 1 1 5B98AB78
-P 5500 4600
-F 0 "D18" H 5500 4700 50  0000 C CNN
-F 1 "GREEN" H 5650 4500 50  0000 R CNN
-F 2 "LED_SMD:LED_0805_2012Metric" H 5500 4600 50  0001 C CNN
-F 3 "http://optoelectronics.liteon.com/upload/download/DS22-2000-073/LTST-C170KGKT.pdf" H 5500 4600 50  0001 C CNN
-F 4 "www.liteon.com" H 5500 4600 60  0001 C CNN "MNF1_URL"
-F 5 "LTST-C170TGKT " H 5500 4600 50  0001 C CNN "MPN"
-F 6 "859-LTST-C170TGKT" H 5500 4600 50  0001 C CNN "Mouser"
-F 7 "160-1887-1-ND" H 5500 4600 50  0001 C CNN "Digikey"
-F 8 "C364562" H 5500 4600 50  0001 C CNN "LCSC"
-F 9 "FV005" H 5500 4600 50  0001 C CNN "Koncar"
-F 10 "T" H 5500 4600 50  0001 C CNN "Side"
-	1    5500 4600
-	1    0    0    -1
-$EndComp
-$Comp
-L power:+3V3 #PWR0122
-U 1 1 5F0C55F7
-P 4250 5850
-F 0 "#PWR0122" H 4250 5700 50  0001 C CNN
-F 1 "+3V3" H 4250 5990 50  0000 C CNN
-F 2 "" H 4250 5850 50  0000 C CNN
-F 3 "" H 4250 5850 50  0000 C CNN
-	1    4250 5850
-	0    -1   -1   0
-$EndComp
 $EndSCHEMATC
