File: SDRAM_JTAG_SD_card_EEPROM.sch (KiCad schematic (older format))
At the start: 21 parts, among them IC6 N.C., IC7 IS42S16400J, IC8 AT24C256C-SSHL-B, J1 503398-1892, X4 N.C.

Commit message: New annotation - All STM32 parts are +100
Changed lines of the file:
@@
 EESchema Schematic File Version 4
-LIBS:ulx3s-cache
-EELAYER 29 0
+EELAYER 30 0
 EELAYER END
 $Descr User 12095 8568
@@
 AR Path="/6720305015B03D7" Ref="J1"  Part="1"
 AR Path="/5F88D5B3/6720305015B03D7" Ref="J1"  Part="1"
-AR Path="/5F8FA164/015B03D7" Ref="J1"  Part="1"
-F 0 "J1" H 10000 5225 59  0000 L BNN
+AR Path="/5F8FA164/015B03D7" Ref="J101"  Part="1"
+F 0 "J101" H 10000 5225 59  0000 L BNN
 F 1 "503398-1892" H 10000 3900 59  0000 L BNN
 F 2 "EEZ DIB MCU r3B4:5033981892" H 10400 4600 50  0001 C CNN
@@
 AR Path="/5478ABB4F3A8FBBF" Ref="IC7"  Part="1"
 AR Path="/5F88D5B3/5478ABB4F3A8FBBF" Ref="IC7"  Part="1"
-AR Path="/5F8FA164/F3A8FBBF" Ref="IC7"  Part="1"
-F 0 "IC7" H 3014 5034 59  0000 L BNN
+AR Path="/5F8FA164/F3A8FBBF" Ref="IC107"  Part="1"
+F 0 "IC107" H 3014 5034 59  0000 L BNN
 F 1 "IS42S16400J" H 2700 1400 59  0000 L BNN
 F 2 "EEZ DIB MCU r3B4:TSOPII-54" H 3200 3300 50  0001 C CNN
@@
 AR Path="/7152EFE5F11CC9BA" Ref="IC6"  Part="1"
 AR Path="/5F88D5B3/7152EFE5F11CC9BA" Ref="IC6"  Part="1"
-AR Path="/5F8FA164/F11CC9BA" Ref="IC6"  Part="1"
-F 0 "IC6" H 6195 1628 69  0000 L BNN
+AR Path="/5F8FA164/F11CC9BA" Ref="IC106"  Part="1"
+F 0 "IC106" H 6195 1628 69  0000 L BNN
 F 1 "N.C." H 5962 993 69  0000 L BNN
 F 2 "EEZ DIB MCU r3B4:DRL6" H 6300 1400 50  0001 C CNN
@@
 AR Path="/8100104B34249FE4" Ref="IC8"  Part="1"
 AR Path="/5F88D5B3/8100104B34249FE4" Ref="IC8"  Part="1"
-AR Path="/5F8FA164/34249FE4" Ref="IC8"  Part="1"
-F 0 "IC8" H 6289 4934 69  0000 L BNN
+AR Path="/5F8FA164/34249FE4" Ref="IC108"  Part="1"
+F 0 "IC108" H 6289 4934 69  0000 L BNN
 F 1 "AT24C256C-SSHL-B" H 5964 4183 69  0000 L BNN
 F 2 "EEZ DIB MCU r3B4:SOIC127P600X173-8N" H 6400 4600 50  0001 C CNN
@@
 AR Path="/B2768A806716FC81" Ref="JP5"  Part="1"
 AR Path="/5F88D5B3/B2768A806716FC81" Ref="JP5"  Part="1"
-AR Path="/5F8FA164/6716FC81" Ref="JP5"  Part="1"
-F 0 "JP5" H 7650 1850 59  0000 L BNN
+AR Path="/5F8FA164/6716FC81" Ref="JP105"  Part="1"
+F 0 "JP105" H 7650 1850 59  0000 L BNN
 F 1 "JP2-CUT" H 7700 1800 50  0001 C CNN
 F 2 "EEZ DIB MCU r3B4:JP2-CUT" H 7700 1800 50  0001 C CNN
@@
 	1    7500 1800
 	0    -1   1    0
-$EndComp
-$Comp
-L SDRAM_JTAG_SD_card_EEPROM-rescue:SSW-106-02-S-S-EEZ_DIB_MCU_r3B4-eagle-import X4
-U 6 1 8D13266F
-P 8200 2700
-AR Path="/8D73A588D13266F" Ref="X4"  Part="6"
-AR Path="/5F88D5B3/8D73A588D13266F" Ref="X4"  Part="6"
-AR Path="/5F8FA164/8D13266F" Ref="X4"  Part="6"
-F 0 "X4" H 8080 2730 51  0000 R TNN
-F 1 "N.C." H 8100 2800 59  0001 L BNN
-F 2 "EEZ DIB MCU r3B4:SSW-106-02-S-S" H 8200 2700 50  0001 C CNN
-F 3 "" H 8200 2700 50  0001 C CNN
-	6    8200 2700
-	-1   0    0    -1
 $EndComp
 $Comp
@@
 Wire Bus Line
 	4300 1300 4300 3100
+$Comp
+L SDRAM_JTAG_SD_card_EEPROM-rescue:SSW-106-02-S-S-EEZ_DIB_MCU_r3B4-eagle-import X4
+U 6 1 8D13266F
+P 8200 2700
+AR Path="/8D73A588D13266F" Ref="X4"  Part="6"
+AR Path="/5F88D5B3/8D73A588D13266F" Ref="X4"  Part="6"
+AR Path="/5F8FA164/8D13266F" Ref="X4"  Part="6"
+F 0 "X4" H 8080 2730 51  0000 R TNN
+F 1 "N.C." H 8100 2800 59  0001 L BNN
+F 2 "EEZ DIB MCU r3B4:SSW-106-02-S-S" H 8200 2700 50  0001 C CNN
+F 3 "" H 8200 2700 50  0001 C CNN
+	6    8200 2700
+	-1   0    0    -1
+$EndComp
 $EndSCHEMATC

Commit message: Adding default parts
Parts:
- C40, C42, C43, C44, C45, C46, C47, C48, C49: footprint EEZ DIB MCU r3B4:C0603 -> Capacitor_SMD:C_0603_1608Metric
- C41: footprint EEZ DIB MCU r3B4:C1206 -> Capacitor_SMD:C_1206_3216Metric
- IC7: footprint EEZ DIB MCU r3B4:TSOPII-54 -> Package_SO:TSOP-II-54_22.2x10.16mm_P0.8mm
- R19, R20, R21, R22, R23: footprint EEZ DIB MCU r3B4:R0805 -> Resistor_SMD:R_0805_2012Metric
Changed lines of the file:
@@
 F 0 "IC107" H 3014 5034 59  0000 L BNN
 F 1 "IS42S16400J" H 2700 1400 59  0000 L BNN
-F 2 "EEZ DIB MCU r3B4:TSOPII-54" H 3200 3300 50  0001 C CNN
+F 2 "Package_SO:TSOP-II-54_22.2x10.16mm_P0.8mm" H 3200 3300 50  0001 C CNN
 F 3 "" H 3200 3300 50  0001 C CNN
 	1    3200 3300
@@
 F 0 "C143" H 2085 5965 59  0000 L BNN
 F 1 "100n" H 2085 5890 59  0000 L BNN
-F 2 "EEZ DIB MCU r3B4:C0603" H 2000 6000 50  0001 C CNN
+F 2 "Capacitor_SMD:C_0603_1608Metric" H 2000 6000 50  0001 C CNN
 F 3 "" H 2000 6000 50  0001 C CNN
 	1    2000 6000
@@
 F 0 "C144" H 2485 5965 59  0000 L BNN
 F 1 "100n" H 2485 5890 59  0000 L BNN
-F 2 "EEZ DIB MCU r3B4:C0603" H 2400 6000 50  0001 C CNN
+F 2 "Capacitor_SMD:C_0603_1608Metric" H 2400 6000 50  0001 C CNN
 F 3 "" H 2400 6000 50  0001 C CNN
 	1    2400 6000
@@
 F 0 "C145" H 2885 5965 59  0000 L BNN
 F 1 "100n" H 2885 5890 59  0000 L BNN
-F 2 "EEZ DIB MCU r3B4:C0603" H 2800 6000 50  0001 C CNN
+F 2 "Capacitor_SMD:C_0603_1608Metric" H 2800 6000 50  0001 C CNN
 F 3 "" H 2800 6000 50  0001 C CNN
 	1    2800 6000
@@
 F 0 "C146" H 3285 5965 59  0000 L BNN
 F 1 "100n" H 3285 5890 59  0000 L BNN
-F 2 "EEZ DIB MCU r3B4:C0603" H 3200 6000 50  0001 C CNN
+F 2 "Capacitor_SMD:C_0603_1608Metric" H 3200 6000 50  0001 C CNN
 F 3 "" H 3200 6000 50  0001 C CNN
 	1    3200 6000
@@
 F 0 "C147" H 3685 5965 59  0000 L BNN
 F 1 "100n" H 3685 5890 59  0000 L BNN
-F 2 "EEZ DIB MCU r3B4:C0603" H 3600 6000 50  0001 C CNN
+F 2 "Capacitor_SMD:C_0603_1608Metric" H 3600 6000 50  0001 C CNN
 F 3 "" H 3600 6000 50  0001 C CNN
 	1    3600 6000
@@
 F 0 "C148" H 4085 5965 59  0000 L BNN
 F 1 "100n" H 4085 5890 59  0000 L BNN
-F 2 "EEZ DIB MCU r3B4:C0603" H 4000 6000 50  0001 C CNN
+F 2 "Capacitor_SMD:C_0603_1608Metric" H 4000 6000 50  0001 C CNN
 F 3 "" H 4000 6000 50  0001 C CNN
 	1    4000 6000
@@
 F 0 "C142" V 7185 4185 59  0000 L BNN
 F 1 "100n" V 7285 4185 59  0000 L BNN
-F 2 "EEZ DIB MCU r3B4:C0603" H 7200 4200 50  0001 C CNN
+F 2 "Capacitor_SMD:C_0603_1608Metric" H 7200 4200 50  0001 C CNN
 F 3 "" H 7200 4200 50  0001 C CNN
 	1    7200 4200
@@
 F 0 "C141" V 9481 4005 59  0000 R BNN
 F 1 "4u7" V 9581 4005 59  0000 R BNN
-F 2 "EEZ DIB MCU r3B4:C1206" H 9500 4100 50  0001 C CNN
+F 2 "Capacitor_SMD:C_1206_3216Metric" H 9500 4100 50  0001 C CNN
 F 3 "" H 9500 4100 50  0001 C CNN
 	1    9500 4100
@@
 F 0 "C140" H 5785 1340 59  0000 L BNN
 F 1 "N.C." H 5785 1265 59  0000 L BNN
-F 2 "EEZ DIB MCU r3B4:C0603" H 5700 1400 50  0001 C CNN
+F 2 "Capacitor_SMD:C_0603_1608Metric" H 5700 1400 50  0001 C CNN
 F 3 "" H 5700 1400 50  0001 C CNN
 	1    5700 1400
@@
 F 0 "R123" V 8791 4150 59  0000 L BNN
 F 1 "47K" V 8880 4150 59  0000 L BNN
-F 2 "EEZ DIB MCU r3B4:R0805" H 8800 4100 50  0001 C CNN
+F 2 "Resistor_SMD:R_0805_2012Metric" H 8800 4100 50  0001 C CNN
 F 3 "" H 8800 4100 50  0001 C CNN
 	1    8800 4100
@@
 F 0 "R122" V 8691 4150 59  0000 L BNN
 F 1 "47K" V 8780 4150 59  0000 L BNN
-F 2 "EEZ DIB MCU r3B4:R0805" H 8700 4100 50  0001 C CNN
+F 2 "Resistor_SMD:R_0805_2012Metric" H 8700 4100 50  0001 C CNN
 F 3 "" H 8700 4100 50  0001 C CNN
 	1    8700 4100
@@
 F 0 "R120" H 6300 2420 59  0000 R BNN
 F 1 "N.C." H 6525 2420 59  0000 L BNN
-F 2 "EEZ DIB MCU r3B4:R0805" H 6400 2400 50  0001 C CNN
+F 2 "Resistor_SMD:R_0805_2012Metric" H 6400 2400 50  0001 C CNN
 F 3 "" H 6400 2400 50  0001 C CNN
 	1    6400 2400
@@
 F 0 "R121" H 6300 2509 59  0000 R BNN
 F 1 "N.C." H 6525 2520 59  0000 L BNN
-F 2 "EEZ DIB MCU r3B4:R0805" H 6400 2500 50  0001 C CNN
+F 2 "Resistor_SMD:R_0805_2012Metric" H 6400 2500 50  0001 C CNN
 F 3 "" H 6400 2500 50  0001 C CNN
 	1    6400 2500
@@
 F 0 "R119" V 8020 1950 59  0000 R TNN
 F 1 "N.C." V 7920 1950 59  0000 R TNN
-F 2 "EEZ DIB MCU r3B4:R0805" H 8000 2000 50  0001 C CNN
+F 2 "Resistor_SMD:R_0805_2012Metric" H 8000 2000 50  0001 C CNN
 F 3 "" H 8000 2000 50  0001 C CNN
 	1    8000 2000
@@
 F 0 "C149" H 4485 5965 59  0000 L BNN
 F 1 "100n" H 4485 5890 59  0000 L BNN
-F 2 "EEZ DIB MCU r3B4:C0603" H 4400 6000 50  0001 C CNN
+F 2 "Capacitor_SMD:C_0603_1608Metric" H 4400 6000 50  0001 C CNN
 F 3 "" H 4400 6000 50  0001 C CNN
 	1    4400 6000
@@
 Wire Notes Line
 	4800 3200 11000 3200
-Wire Bus Line
-	2100 1500 2100 2800
-Wire Bus Line
-	4300 1300 4300 3100
 $Comp
 L SDRAM_JTAG_SD_card_EEPROM-rescue:SSW-106-02-S-S-EEZ_DIB_MCU_r3B4-eagle-import X4
@@
 	-1   0    0    -1
 $EndComp
+Wire Bus Line
+	2100 1500 2100 2800
+Wire Bus Line
+	4300 1300 4300 3100
 $EndSCHEMATC

Commit message: Adding TO FROM FPGA lines
Connections:
- net labels added: SDMMC1_FROM_FPGA_CK, SDMMC1_FROM_FPGA_CMD, SDMMC1_FROM_FPGA_D0, SD_FROM_FPGA_DETECT
- net labels removed: SDMMC1_CK, SDMMC1_CMD, SDMMC1_D0, SD_DETECT
Changed lines of the file:
@@
 Wire Wire Line
 	2600 4200 2000 4200
-Text GLabel 2000 4200 2    50   BiDi ~ 0
+Text GLabel 2000 4200 0    50   BiDi ~ 0
 FMC_SDNRAS
 Wire Wire Line
 	2600 4300 2000 4300
-Text GLabel 2000 4300 2    50   BiDi ~ 0
+Text GLabel 2000 4300 0    50   BiDi ~ 0
 FMC_SDNCAS
 Wire Wire Line
 	2600 4400 2000 4400
-Text GLabel 2000 4400 2    50   BiDi ~ 0
+Text GLabel 2000 4400 0    50   BiDi ~ 0
 FMC_SDNWE
 Wire Wire Line
 	2600 4500 2000 4500
-Text GLabel 2000 4500 2    50   BiDi ~ 0
+Text GLabel 2000 4500 0    50   BiDi ~ 0
 FMC_SDNE0
 Wire Wire Line
@@
 Wire Wire Line
 	2600 3100 2000 3100
-Text GLabel 2000 3100 2    50   BiDi ~ 0
+Text GLabel 2000 3100 0    50   BiDi ~ 0
 FMC_BA0
 Wire Wire Line
 	2600 3200 2000 3200
-Text GLabel 2000 3200 2    50   BiDi ~ 0
+Text GLabel 2000 3200 0    50   BiDi ~ 0
 FMC_BA1
 Wire Wire Line
@@
 Wire Wire Line
 	2600 3700 2000 3700
-Text GLabel 2000 3700 2    50   BiDi ~ 0
+Text GLabel 2000 3700 0    50   BiDi ~ 0
 FMC_NBL1
 Wire Wire Line
 	2600 3800 2000 3800
-Text GLabel 2000 3800 2    50   BiDi ~ 0
+Text GLabel 2000 3800 0    50   BiDi ~ 0
 FMC_NBL0
 Wire Wire Line
 	2600 5000 2000 5000
-Text GLabel 2000 5000 2    50   BiDi ~ 0
+Text GLabel 2000 5000 0    50   BiDi ~ 0
 FMC_SDCKE0
 Wire Wire Line
 	2600 4900 2000 4900
-Text GLabel 2000 4900 2    50   BiDi ~ 0
+Text GLabel 2000 4900 0    50   BiDi ~ 0
 FMC_SDCLK
 Wire Wire Line
@@
 Wire Wire Line
 	5900 4500 5300 4500
-Text GLabel 5300 4500 2    50   BiDi ~ 0
+Text GLabel 5300 4500 0    50   BiDi ~ 0
 I2C1_SDA
 Wire Wire Line
 	5900 4400 5300 4400
-Text GLabel 5300 4400 2    50   BiDi ~ 0
+Text GLabel 5300 4400 0    50   BiDi ~ 0
 I2C1_SCL
 Wire Wire Line
 	9900 5100 8000 5100
 Text GLabel 8000 5100 2    50   BiDi ~ 0
-SD_DETECT
-Wire Wire Line
-	8700 4800 8000 4800
-Wire Wire Line
-	8700 4300 8700 4800
+SD_FROM_FPGA_DETECT
 Wire Wire Line
 	8700 4800 9900 4800
-Text GLabel 8000 4800 2    50   BiDi ~ 0
-SDMMC1_D0
-Connection ~ 8700 4800
-Wire Wire Line
-	8800 4400 8000 4400
 Wire Wire Line
 	8800 4300 8800 4400
 Wire Wire Line
 	9900 4400 8800 4400
-Text GLabel 8000 4400 2    50   BiDi ~ 0
-SDMMC1_CMD
-Connection ~ 8800 4400
-Wire Wire Line
-	8000 4600 9900 4600
-Text GLabel 8000 4600 2    50   BiDi ~ 0
-SDMMC1_CK
 Wire Wire Line
 	8100 2400 7100 2400
@@
 	-1   0    0    -1
 $EndComp
+Connection ~ 8700 4800
+Wire Wire Line
+	8700 4800 8000 4800
+Wire Wire Line
+	8000 4600 9900 4600
+Wire Wire Line
+	8700 4300 8700 4800
+Wire Bus Line
+	4300 1300 4300 3100
 Wire Bus Line
 	2100 1500 2100 2800
-Wire Bus Line
-	4300 1300 4300 3100
+Connection ~ 8800 4400
+Wire Wire Line
+	8800 4400 8000 4400
+Text GLabel 8000 4400 2    50   BiDi ~ 0
+SDMMC1_FROM_FPGA_CMD
+Text GLabel 8000 4800 2    50   BiDi ~ 0
+SDMMC1_FROM_FPGA_D0
+Text GLabel 8000 4600 2    50   BiDi ~ 0
+SDMMC1_FROM_FPGA_CK
 $EndSCHEMATC

Commit message: Rewiering LCD OUT to bottom left
Parts:
- R22, R23: footprint Resistor_SMD:R_0805_2012Metric -> Resistor_SMD:R_0603_1608Metric
Changed lines of the file:
@@
 F 0 "R123" V 8791 4150 59  0000 L BNN
 F 1 "47K" V 8880 4150 59  0000 L BNN
-F 2 "Resistor_SMD:R_0805_2012Metric" H 8800 4100 50  0001 C CNN
+F 2 "Resistor_SMD:R_0603_1608Metric" H 8800 4100 50  0001 C CNN
 F 3 "" H 8800 4100 50  0001 C CNN
 	1    8800 4100
@@
 F 0 "R122" V 8691 4150 59  0000 L BNN
 F 1 "47K" V 8780 4150 59  0000 L BNN
-F 2 "Resistor_SMD:R_0805_2012Metric" H 8700 4100 50  0001 C CNN
+F 2 "Resistor_SMD:R_0603_1608Metric" H 8700 4100 50  0001 C CNN
 F 3 "" H 8700 4100 50  0001 C CNN
 	1    8700 4100
