File: SDRAM_JTAG_SD_card_EEPROM.sch (KiCad schematic (older format))
At the start: 21 parts, among them IC6 N.C., IC7 IS42S16400J, IC8 AT24C256C-SSHL-B, J1 503398-1892, X4 N.C.

Commit message: More schematics cleanup
Connections:
- net labels removed: FMC_A[0..12], FMC_D[0..15]
