File: Ethernet_PHY.sch (KiCad schematic (older format))
At the start: 44 parts, among them IC13 N.C., IC14 DP83848CVV_NOPB, X5 LMJTAB881243M-L

Commit message: All STM32 parts are now +100, moving parts to original position
Changed lines of the file:
@@
 AR Path="/5F88DC09/F6EC8A3AAF5BEB10" Ref="C62"  Part="1"
 AR Path="/5F8FF86F/F6EC8A3AAF5BEB10" Ref="C62"  Part="1"
-AR Path="/5F8FF86F/AF5BEB10" Ref="C62"  Part="1"
-F 0 "C62" V 7215 3215 59  0000 R TNN
+AR Path="/5F8FF86F/AF5BEB10" Ref="C162"  Part="1"
+F 0 "C162" V 7215 3215 59  0000 R TNN
 F 1 "100n" V 7315 3215 59  0000 R TNN
 F 2 "EEZ DIB MCU r3B4:C0603" H 7300 3300 50  0001 C CNN
@@
 AR Path="/5F88DC09/761E0343A6258458" Ref="JP8"  Part="1"
 AR Path="/5F8FF86F/761E0343A6258458" Ref="JP8"  Part="1"
-AR Path="/5F8FF86F/A6258458" Ref="JP8"  Part="1"
-F 0 "JP8" V 1900 3425 59  0000 L TNN
+AR Path="/5F8FF86F/A6258458" Ref="JP108"  Part="1"
+F 0 "JP108" V 1900 3425 59  0000 L TNN
 F 1 "JP2-CUT" H 1900 3400 50  0001 C CNN
 F 2 "EEZ DIB MCU r3B4:JP2-CUT" H 1900 3400 50  0001 C CNN
@@
 AR Path="/5F88DC09/8E0DE4F6E957C24B" Ref="JP9"  Part="1"
 AR Path="/5F8FF86F/8E0DE4F6E957C24B" Ref="JP9"  Part="1"
-AR Path="/5F8FF86F/E957C24B" Ref="JP9"  Part="1"
-F 0 "JP9" V 2000 3375 59  0000 R TNN
+AR Path="/5F8FF86F/E957C24B" Ref="JP109"  Part="1"
+F 0 "JP109" V 2000 3375 59  0000 R TNN
 F 1 "JP2-CUT" H 2000 3400 50  0001 C CNN
 F 2 "EEZ DIB MCU r3B4:JP2-CUT" H 2000 3400 50  0001 C CNN
@@
 AR Path="/5F88DC09/4ADB8E0A33F1B700" Ref="JP10"  Part="1"
 AR Path="/5F8FF86F/4ADB8E0A33F1B700" Ref="JP10"  Part="1"
-AR Path="/5F8FF86F/33F1B700" Ref="JP10"  Part="1"
-F 0 "JP10" V 3000 3375 59  0000 R TNN
+AR Path="/5F8FF86F/33F1B700" Ref="JP110"  Part="1"
+F 0 "JP110" V 3000 3375 59  0000 R TNN
 F 1 "JP2-CUT" H 3000 3400 50  0001 C CNN
 F 2 "EEZ DIB MCU r3B4:JP2-CUT" H 3000 3400 50  0001 C CNN
@@
 AR Path="/5F88DC09/BD05527201682B0F" Ref="JP12"  Part="1"
 AR Path="/5F8FF86F/BD05527201682B0F" Ref="JP12"  Part="1"
-AR Path="/5F8FF86F/01682B0F" Ref="JP12"  Part="1"
-F 0 "JP12" H 2725 4900 59  0000 L BNN
+AR Path="/5F8FF86F/01682B0F" Ref="JP112"  Part="1"
+F 0 "JP112" H 2725 4900 59  0000 L BNN
 F 1 "JP2-NOCUT" H 2800 5000 50  0001 C CNN
 F 2 "EEZ DIB MCU r3B4:JP2-NOCUT" H 2800 5000 50  0001 C CNN
@@
 AR Path="/5F88DC09/F74C9D7641450E5" Ref="JP11"  Part="1"
 AR Path="/5F8FF86F/F74C9D7641450E5" Ref="JP11"  Part="1"
-AR Path="/5F8FF86F/641450E5" Ref="JP11"  Part="1"
-F 0 "JP11" H 1925 3600 59  0000 R BNN
+AR Path="/5F8FF86F/641450E5" Ref="JP111"  Part="1"
+F 0 "JP111" H 1925 3600 59  0000 R BNN
 F 1 "JP2-NOCUT" H 1800 3700 50  0001 C CNN
 F 2 "EEZ DIB MCU r3B4:JP2-NOCUT" H 1800 3700 50  0001 C CNN

Commit message: Adding default parts
Parts:
- C59, C60, C61, C62, C63, C64, C65, C67, C68, C69, C70: footprint EEZ DIB MCU r3B4:C0603 -> Capacitor_SMD:C_0603_1608Metric
- C66: footprint EEZ DIB MCU r3B4:EC1206 -> Capacitor_SMD:C_1206_3216Metric
- R34, R35, R36, R37, R38, R39, R40, R41, R42, R43, R44, R45, R46, R47, R48, R49, R50, R51: footprint EEZ DIB MCU r3B4:R0805 -> Resistor_SMD:R_0805_2012Metric
Changed lines of the file:
@@
 F 0 "R148" V 5480 4750 59  0000 L BNN
 F 1 "2K2" V 5405 4750 59  0000 L BNN
-F 2 "EEZ DIB MCU r3B4:R0805" H 5400 4700 50  0001 C CNN
+F 2 "Resistor_SMD:R_0805_2012Metric" H 5400 4700 50  0001 C CNN
 F 3 "" H 5400 4700 50  0001 C CNN
 	1    5400 4700
@@
 F 0 "R149" V 5520 4650 59  0000 R TNN
 F 1 "2K2" V 5445 4650 59  0000 R TNN
-F 2 "EEZ DIB MCU r3B4:R0805" H 5500 4700 50  0001 C CNN
+F 2 "Resistor_SMD:R_0805_2012Metric" H 5500 4700 50  0001 C CNN
 F 3 "" H 5500 4700 50  0001 C CNN
 	1    5500 4700
@@
 F 0 "C164" H 5715 4735 59  0000 R TNN
 F 1 "100n" H 5715 4660 59  0000 R TNN
-F 2 "EEZ DIB MCU r3B4:C0603" H 5800 4700 50  0001 C CNN
+F 2 "Capacitor_SMD:C_0603_1608Metric" H 5800 4700 50  0001 C CNN
 F 3 "" H 5800 4700 50  0001 C CNN
 	1    5800 4700
@@
 F 0 "C165" H 6115 4735 59  0000 R TNN
 F 1 "100n" H 6115 4660 59  0000 R TNN
-F 2 "EEZ DIB MCU r3B4:C0603" H 6200 4700 50  0001 C CNN
+F 2 "Capacitor_SMD:C_0603_1608Metric" H 6200 4700 50  0001 C CNN
 F 3 "" H 6200 4700 50  0001 C CNN
 	1    6200 4700
@@
 F 0 "R150" V 7395 4650 59  0000 R TNN
 F 1 "4K87" V 7320 4650 59  0000 R TNN
-F 2 "EEZ DIB MCU r3B4:R0805" H 7400 4700 50  0001 C CNN
+F 2 "Resistor_SMD:R_0805_2012Metric" H 7400 4700 50  0001 C CNN
 F 3 "" H 7400 4700 50  0001 C CNN
 	1    7400 4700
@@
 F 0 "C166" H 6505 4725 59  0000 R TNN
 F 1 "10u" H 6505 4640 59  0000 R TNN
-F 2 "EEZ DIB MCU r3B4:EC1206" H 6600 4700 50  0001 C CNN
+F 2 "Capacitor_SMD:C_1206_3216Metric" H 6600 4700 50  0001 C CNN
 F 3 "" H 6600 4700 50  0001 C CNN
 	1    6600 4700
@@
 F 0 "C167" H 6915 4710 59  0000 R TNN
 F 1 "100n" H 6915 4635 59  0000 R TNN
-F 2 "EEZ DIB MCU r3B4:C0603" H 7000 4700 50  0001 C CNN
+F 2 "Capacitor_SMD:C_0603_1608Metric" H 7000 4700 50  0001 C CNN
 F 3 "" H 7000 4700 50  0001 C CNN
 	1    7000 4700
@@
 F 0 "C170" H 2815 5810 59  0000 R TNN
 F 1 "100n" H 2815 5735 59  0000 R TNN
-F 2 "EEZ DIB MCU r3B4:C0603" H 2900 5800 50  0001 C CNN
+F 2 "Capacitor_SMD:C_0603_1608Metric" H 2900 5800 50  0001 C CNN
 F 3 "" H 2900 5800 50  0001 C CNN
 	1    2900 5800
@@
 F 0 "C169" H 2415 5810 59  0000 R TNN
 F 1 "100n" H 2415 5735 59  0000 R TNN
-F 2 "EEZ DIB MCU r3B4:C0603" H 2500 5800 50  0001 C CNN
+F 2 "Capacitor_SMD:C_0603_1608Metric" H 2500 5800 50  0001 C CNN
 F 3 "" H 2500 5800 50  0001 C CNN
 	1    2500 5800
@@
 F 0 "C168" H 2185 5665 59  0000 L BNN
 F 1 "100n" H 2185 5590 59  0000 L BNN
-F 2 "EEZ DIB MCU r3B4:C0603" H 2100 5700 50  0001 C CNN
+F 2 "Capacitor_SMD:C_0603_1608Metric" H 2100 5700 50  0001 C CNN
 F 3 "" H 2100 5700 50  0001 C CNN
 	1    2100 5700
@@
 F 0 "R135" V 7720 2150 59  0000 R TNN
 F 1 "49R9" V 7620 2150 59  0000 R TNN
-F 2 "EEZ DIB MCU r3B4:R0805" H 7700 2200 50  0001 C CNN
+F 2 "Resistor_SMD:R_0805_2012Metric" H 7700 2200 50  0001 C CNN
 F 3 "" H 7700 2200 50  0001 C CNN
 	1    7700 2200
@@
 F 0 "R136" V 7720 2650 59  0000 L TNN
 F 1 "49R9" V 7620 2650 59  0000 L TNN
-F 2 "EEZ DIB MCU r3B4:R0805" H 7700 2600 50  0001 C CNN
+F 2 "Resistor_SMD:R_0805_2012Metric" H 7700 2600 50  0001 C CNN
 F 3 "" H 7700 2600 50  0001 C CNN
 	1    7700 2600
@@
 F 0 "R139" V 7120 3050 59  0000 R TNN
 F 1 "49R9" V 7020 3050 59  0000 R TNN
-F 2 "EEZ DIB MCU r3B4:R0805" H 7100 3100 50  0001 C CNN
+F 2 "Resistor_SMD:R_0805_2012Metric" H 7100 3100 50  0001 C CNN
 F 3 "" H 7100 3100 50  0001 C CNN
 	1    7100 3100
@@
 F 0 "R144" V 7120 3450 59  0000 R TNN
 F 1 "49R9" V 7020 3450 59  0000 R TNN
-F 2 "EEZ DIB MCU r3B4:R0805" H 7100 3500 50  0001 C CNN
+F 2 "Resistor_SMD:R_0805_2012Metric" H 7100 3500 50  0001 C CNN
 F 3 "" H 7100 3500 50  0001 C CNN
 	1    7100 3500
@@
 F 0 "C160" V 7415 2315 59  0000 R TNN
 F 1 "100n" V 7515 2315 59  0000 R TNN
-F 2 "EEZ DIB MCU r3B4:C0603" H 7500 2400 50  0001 C CNN
+F 2 "Capacitor_SMD:C_0603_1608Metric" H 7500 2400 50  0001 C CNN
 F 3 "" H 7500 2400 50  0001 C CNN
 	1    7500 2400
@@
 F 0 "C162" V 7215 3215 59  0000 R TNN
 F 1 "100n" V 7315 3215 59  0000 R TNN
-F 2 "EEZ DIB MCU r3B4:C0603" H 7300 3300 50  0001 C CNN
+F 2 "Capacitor_SMD:C_0603_1608Metric" H 7300 3300 50  0001 C CNN
 F 3 "" H 7300 3300 50  0001 C CNN
 	1    7300 3300
@@
 F 0 "R138" H 6600 3055 59  0000 R TNN
 F 1 "2K2" H 6375 3080 59  0000 R TNN
-F 2 "EEZ DIB MCU r3B4:R0805" H 6500 3100 50  0001 C CNN
+F 2 "Resistor_SMD:R_0805_2012Metric" H 6500 3100 50  0001 C CNN
 F 3 "" H 6500 3100 50  0001 C CNN
 	1    6500 3100
@@
 F 0 "R141" H 6600 3255 59  0000 R TNN
 F 1 "N.C." H 6375 3280 59  0000 R TNN
-F 2 "EEZ DIB MCU r3B4:R0805" H 6500 3300 50  0001 C CNN
+F 2 "Resistor_SMD:R_0805_2012Metric" H 6500 3300 50  0001 C CNN
 F 3 "" H 6500 3300 50  0001 C CNN
 	1    6500 3300
@@
 F 0 "R145" H 6600 3655 59  0000 R TNN
 F 1 "2K2" H 6375 3680 59  0000 R TNN
-F 2 "EEZ DIB MCU r3B4:R0805" H 6500 3700 50  0001 C CNN
+F 2 "Resistor_SMD:R_0805_2012Metric" H 6500 3700 50  0001 C CNN
 F 3 "" H 6500 3700 50  0001 C CNN
 	1    6500 3700
@@
 F 0 "R143" H 6600 3455 59  0000 R TNN
 F 1 "2K2" H 6375 3480 59  0000 R TNN
-F 2 "EEZ DIB MCU r3B4:R0805" H 6500 3500 50  0001 C CNN
+F 2 "Resistor_SMD:R_0805_2012Metric" H 6500 3500 50  0001 C CNN
 F 3 "" H 6500 3500 50  0001 C CNN
 	1    6500 3500
@@
 F 0 "C163" V 8185 3310 59  0000 L BNN
 F 1 "100n" V 8285 3285 59  0000 L BNN
-F 2 "EEZ DIB MCU r3B4:C0603" H 8200 3300 50  0001 C CNN
+F 2 "Capacitor_SMD:C_0603_1608Metric" H 8200 3300 50  0001 C CNN
 F 3 "" H 8200 3300 50  0001 C CNN
 	1    8200 3300
@@
 F 0 "R147" H 6800 3980 59  0000 R TNN
 F 1 "220R" H 6375 3980 59  0000 R TNN
-F 2 "EEZ DIB MCU r3B4:R0805" H 6500 4000 50  0001 C CNN
+F 2 "Resistor_SMD:R_0805_2012Metric" H 6500 4000 50  0001 C CNN
 F 3 "" H 6500 4000 50  0001 C CNN
 	1    6500 4000
@@
 F 0 "R146" H 6800 3880 59  0000 R TNN
 F 1 "220R" H 6375 3880 59  0000 R TNN
-F 2 "EEZ DIB MCU r3B4:R0805" H 6500 3900 50  0001 C CNN
+F 2 "Resistor_SMD:R_0805_2012Metric" H 6500 3900 50  0001 C CNN
 F 3 "" H 6500 3900 50  0001 C CNN
 	1    6500 3900
@@
 F 0 "C161" V 8185 2485 59  0000 L BNN
 F 1 "100n" V 8285 2485 59  0000 L BNN
-F 2 "EEZ DIB MCU r3B4:C0603" H 8200 2500 50  0001 C CNN
+F 2 "Capacitor_SMD:C_0603_1608Metric" H 8200 2500 50  0001 C CNN
 F 3 "" H 8200 2500 50  0001 C CNN
 	1    8200 2500
@@
 F 0 "R140" H 1475 3180 59  0000 R TNN
 F 1 "N.C." H 1725 3180 59  0000 L TNN
-F 2 "EEZ DIB MCU r3B4:R0805" H 1600 3200 50  0001 C CNN
+F 2 "Resistor_SMD:R_0805_2012Metric" H 1600 3200 50  0001 C CNN
 F 3 "" H 1600 3200 50  0001 C CNN
 	1    1600 3200
@@
 F 0 "R142" H 2725 3620 59  0000 L BNN
 F 1 "N.C." H 2725 3545 59  0000 L BNN
-F 2 "EEZ DIB MCU r3B4:R0805" H 2800 3500 50  0001 C CNN
+F 2 "Resistor_SMD:R_0805_2012Metric" H 2800 3500 50  0001 C CNN
 F 3 "" H 2800 3500 50  0001 C CNN
 	1    2800 3500
@@
 F 0 "R137" H 1475 2980 59  0000 R TNN
 F 1 "N.C." H 1725 2980 59  0000 L TNN
-F 2 "EEZ DIB MCU r3B4:R0805" H 1600 3000 50  0001 C CNN
+F 2 "Resistor_SMD:R_0805_2012Metric" H 1600 3000 50  0001 C CNN
 F 3 "" H 1600 3000 50  0001 C CNN
 	1    1600 3000
@@
 F 0 "R151" H 2275 4980 59  0000 R TNN
 F 1 "2K2" H 2325 5130 59  0000 L TNN
-F 2 "EEZ DIB MCU r3B4:R0805" H 2400 5000 50  0001 C CNN
+F 2 "Resistor_SMD:R_0805_2012Metric" H 2400 5000 50  0001 C CNN
 F 3 "" H 2400 5000 50  0001 C CNN
 	1    2400 5000
@@
 F 0 "R134" V 3155 1950 59  0000 L BNN
 F 1 "1K5" V 2995 1950 59  0000 L TNN
-F 2 "EEZ DIB MCU r3B4:R0805" H 3100 1900 50  0001 C CNN
+F 2 "Resistor_SMD:R_0805_2012Metric" H 3100 1900 50  0001 C CNN
 F 3 "" H 3100 1900 50  0001 C CNN
 	1    3100 1900
@@
 F 0 "C159" H 7485 1265 59  0000 L BNN
 F 1 "N.C." H 7485 1165 59  0000 L BNN
-F 2 "EEZ DIB MCU r3B4:C0603" H 7400 1300 50  0001 C CNN
+F 2 "Capacitor_SMD:C_0603_1608Metric" H 7400 1300 50  0001 C CNN
 F 3 "" H 7400 1300 50  0001 C CNN
 	1    7400 1300

Commit message: Rewiering LCD OUT to bottom left
Parts:
- removed C66: 10u, Capacitor_SMD:C_1206_3216Metric, symbol Ethernet_PHY-rescue:ECAP1206-EEZ_DIB_MCU_r3B4-eagle-import
- added C166: 10uF, Capacitor_Tantalum_SMD:CP_EIA-3216-10_Kemet-I, symbol antena:CP_Small
- R37, R46, R47: footprint Resistor_SMD:R_0805_2012Metric -> Resistor_SMD:R_0603_1608Metric
Changed lines of the file:
@@
 	7400 5000 7000 5000
-Wire Wire Line
-	6600 4900 6600 5000
 Wire Wire Line
 	7000 4900 7000 5000
@@
 $EndComp
 $Comp
-L Ethernet_PHY-rescue:ECAP1206-EEZ_DIB_MCU_r3B4-eagle-import C66
-U 1 1 AC9801A5
-P 6600 4700
-AR Path="/84B828EFAC9801A5" Ref="C66"  Part="1"
-AR Path="/5F88DC09/84B828EFAC9801A5" Ref="C66"  Part="1"
-AR Path="/5F8FF86F/84B828EFAC9801A5" Ref="C66"  Part="1"
-AR Path="/5F8FF86F/AC9801A5" Ref="C166"  Part="1"
-F 0 "C166" H 6505 4725 59  0000 R TNN
-F 1 "10u" H 6505 4640 59  0000 R TNN
-F 2 "Capacitor_SMD:C_1206_3216Metric" H 6600 4700 50  0001 C CNN
-F 3 "" H 6600 4700 50  0001 C CNN
-	1    6600 4700
-	-1   0    0    -1
-$EndComp
-$Comp
 L Ethernet_PHY-rescue:C-EUC0603-EEZ_DIB_MCU_r3B4-eagle-import C67
 U 1 1 7D1C0DDE
@@
 F 0 "R147" H 6800 3980 59  0000 R TNN
 F 1 "220R" H 6375 3980 59  0000 R TNN
-F 2 "Resistor_SMD:R_0805_2012Metric" H 6500 4000 50  0001 C CNN
+F 2 "Resistor_SMD:R_0603_1608Metric" H 6500 4000 50  0001 C CNN
 F 3 "" H 6500 4000 50  0001 C CNN
 	1    6500 4000
@@
 F 0 "R146" H 6800 3880 59  0000 R TNN
 F 1 "220R" H 6375 3880 59  0000 R TNN
-F 2 "Resistor_SMD:R_0805_2012Metric" H 6500 3900 50  0001 C CNN
+F 2 "Resistor_SMD:R_0603_1608Metric" H 6500 3900 50  0001 C CNN
 F 3 "" H 6500 3900 50  0001 C CNN
 	1    6500 3900
@@
 F 0 "R137" H 1475 2980 59  0000 R TNN
 F 1 "N.C." H 1725 2980 59  0000 L TNN
-F 2 "Resistor_SMD:R_0805_2012Metric" H 1600 3000 50  0001 C CNN
+F 2 "Resistor_SMD:R_0603_1608Metric" H 1600 3000 50  0001 C CNN
 F 3 "" H 1600 3000 50  0001 C CNN
 	1    1600 3000
@@
 AR Path="/5F88DC09/92356C4F5996E8C1" Ref="RN5"  Part="4"
 AR Path="/5F8FF86F/92356C4F5996E8C1" Ref="RN5"  Part="4"
-AR Path="/5F8FF86F/5996E8C1" Ref="RN5"  Part="4"
-F 0 "RN5" H 2200 3705 59  0000 R BNN
+AR Path="/5F8FF86F/5996E8C1" Ref="RN105"  Part="4"
+F 0 "RN105" H 2200 3705 59  0000 R BNN
 F 1 "DR1206-33R-4/8" H 2600 3705 59  0000 L BNN
 F 2 "EEZ DIB MCU r3B4:CAY16" H 2400 3700 50  0001 C CNN
@@
 AR Path="/5F88DC09/92356C4F5996E8D5" Ref="RN5"  Part="1"
 AR Path="/5F8FF86F/92356C4F5996E8D5" Ref="RN5"  Part="1"
-AR Path="/5F8FF86F/5996E8D5" Ref="RN5"  Part="1"
-F 0 "RN5" H 2200 3605 59  0000 R BNN
+AR Path="/5F8FF86F/5996E8D5" Ref="RN105"  Part="1"
+F 0 "RN105" H 2200 3605 59  0000 R BNN
 F 1 "DR1206-33R-4/8" H 2500 3480 59  0001 L BNN
 F 2 "EEZ DIB MCU r3B4:CAY16" H 2400 3600 50  0001 C CNN
@@
 AR Path="/5F88DC09/92356C4F5996E8D9" Ref="RN5"  Part="2"
 AR Path="/5F8FF86F/92356C4F5996E8D9" Ref="RN5"  Part="2"
-AR Path="/5F8FF86F/5996E8D9" Ref="RN5"  Part="2"
-F 0 "RN5" H 2200 4105 59  0000 R BNN
+AR Path="/5F8FF86F/5996E8D9" Ref="RN105"  Part="2"
+F 0 "RN105" H 2200 4105 59  0000 R BNN
 F 1 "DR1206-33R-4/8" H 2500 3980 59  0001 L BNN
 F 2 "EEZ DIB MCU r3B4:CAY16" H 2400 4100 50  0001 C CNN
@@
 AR Path="/5F88DC09/92356C4F5996E8DD" Ref="RN5"  Part="3"
 AR Path="/5F8FF86F/92356C4F5996E8DD" Ref="RN5"  Part="3"
-AR Path="/5F8FF86F/5996E8DD" Ref="RN5"  Part="3"
-F 0 "RN5" H 2200 4205 59  0000 R BNN
+AR Path="/5F8FF86F/5996E8DD" Ref="RN105"  Part="3"
+F 0 "RN105" H 2200 4205 59  0000 R BNN
 F 1 "DR1206-33R-4/8" H 2500 4080 59  0001 L BNN
 F 2 "EEZ DIB MCU r3B4:CAY16" H 2400 4200 50  0001 C CNN
@@
 AR Path="/5F88DC09/893038F797A67697" Ref="RN7"  Part="4"
 AR Path="/5F8FF86F/893038F797A67697" Ref="RN7"  Part="4"
-AR Path="/5F8FF86F/97A67697" Ref="RN7"  Part="4"
-F 0 "RN7" H 2200 4605 59  0000 R BNN
+AR Path="/5F8FF86F/97A67697" Ref="RN107"  Part="4"
+F 0 "RN107" H 2200 4605 59  0000 R BNN
 F 1 "DR1206-33R-4/8" H 2600 4605 59  0000 L BNN
 F 2 "EEZ DIB MCU r3B4:CAY16" H 2400 4600 50  0001 C CNN
@@
 AR Path="/5F88DC09/893038F797A67683" Ref="RN7"  Part="1"
 AR Path="/5F8FF86F/893038F797A67683" Ref="RN7"  Part="1"
-AR Path="/5F8FF86F/97A67683" Ref="RN7"  Part="1"
-F 0 "RN7" H 2200 4705 59  0000 R BNN
+AR Path="/5F8FF86F/97A67683" Ref="RN107"  Part="1"
+F 0 "RN107" H 2200 4705 59  0000 R BNN
 F 1 "DR1206-33R-4/8" H 2500 4580 59  0001 L BNN
 F 2 "EEZ DIB MCU r3B4:CAY16" H 2400 4700 50  0001 C CNN
@@
 AR Path="/5F88DC09/893038F797A6768F" Ref="RN7"  Part="2"
 AR Path="/5F8FF86F/893038F797A6768F" Ref="RN7"  Part="2"
-AR Path="/5F8FF86F/97A6768F" Ref="RN7"  Part="2"
-F 0 "RN7" H 2200 4805 59  0000 R BNN
+AR Path="/5F8FF86F/97A6768F" Ref="RN107"  Part="2"
+F 0 "RN107" H 2200 4805 59  0000 R BNN
 F 1 "DR1206-33R-4/8" H 2500 4680 59  0001 L BNN
 F 2 "EEZ DIB MCU r3B4:CAY16" H 2400 4800 50  0001 C CNN
@@
 AR Path="/5F88DC09/893038F797A6768B" Ref="RN7"  Part="3"
 AR Path="/5F8FF86F/893038F797A6768B" Ref="RN7"  Part="3"
-AR Path="/5F8FF86F/97A6768B" Ref="RN7"  Part="3"
-F 0 "RN7" H 2200 4905 59  0000 R BNN
+AR Path="/5F8FF86F/97A6768B" Ref="RN107"  Part="3"
+F 0 "RN107" H 2200 4905 59  0000 R BNN
 F 1 "DR1206-33R-4/8" H 2500 4780 59  0001 L BNN
 F 2 "EEZ DIB MCU r3B4:CAY16" H 2400 4900 50  0001 C CNN
@@
 AR Path="/5F88DC09/D4DDA4C0A119EF8F" Ref="RN4"  Part="3"
 AR Path="/5F8FF86F/D4DDA4C0A119EF8F" Ref="RN4"  Part="3"
-AR Path="/5F8FF86F/A119EF8F" Ref="RN4"  Part="3"
-F 0 "RN4" H 2200 3905 59  0000 R BNN
+AR Path="/5F8FF86F/A119EF8F" Ref="RN104"  Part="3"
+F 0 "RN104" H 2200 3905 59  0000 R BNN
 F 1 "DR1206-33R-4/8" H 2500 3780 59  0001 L BNN
 F 2 "EEZ DIB MCU r3B4:CAY16" H 2400 3900 50  0001 C CNN
@@
 AR Path="/5F88DC09/FDCEADBA97F649F8" Ref="RN6"  Part="4"
 AR Path="/5F8FF86F/FDCEADBA97F649F8" Ref="RN6"  Part="4"
-AR Path="/5F8FF86F/97F649F8" Ref="RN6"  Part="4"
-F 0 "RN6" H 2200 4305 59  0000 R BNN
+AR Path="/5F8FF86F/97F649F8" Ref="RN106"  Part="4"
+F 0 "RN106" H 2200 4305 59  0000 R BNN
 F 1 "DR1206-33R-4/8" H 2600 4305 59  0000 L BNN
 F 2 "EEZ DIB MCU r3B4:CAY16" H 2400 4300 50  0001 C CNN
@@
 AR Path="/5F88DC09/FDCEADBA97F649EC" Ref="RN6"  Part="1"
 AR Path="/5F8FF86F/FDCEADBA97F649EC" Ref="RN6"  Part="1"
-AR Path="/5F8FF86F/97F649EC" Ref="RN6"  Part="1"
-F 0 "RN6" H 2200 4405 59  0000 R BNN
+AR Path="/5F8FF86F/97F649EC" Ref="RN106"  Part="1"
+F 0 "RN106" H 2200 4405 59  0000 R BNN
 F 1 "DR1206-33R-4/8" H 2500 4280 59  0001 L BNN
 F 2 "EEZ DIB MCU r3B4:CAY16" H 2400 4400 50  0001 C CNN
@@
 AR Path="/5F88DC09/D4DDA4C0A119EF8B" Ref="RN4"  Part="2"
 AR Path="/5F8FF86F/D4DDA4C0A119EF8B" Ref="RN4"  Part="2"
-AR Path="/5F8FF86F/A119EF8B" Ref="RN4"  Part="2"
-F 0 "RN4" H 2000 2805 59  0000 R BNN
+AR Path="/5F8FF86F/A119EF8B" Ref="RN104"  Part="2"
+F 0 "RN104" H 2000 2805 59  0000 R BNN
 F 1 "DR1206-33R-4/8" H 2300 2680 59  0001 L BNN
 F 2 "EEZ DIB MCU r3B4:CAY16" H 2200 2800 50  0001 C CNN
@@
 AR Path="/5F88DC09/D4DDA4C0A119EF87" Ref="RN4"  Part="1"
 AR Path="/5F8FF86F/D4DDA4C0A119EF87" Ref="RN4"  Part="1"
-AR Path="/5F8FF86F/A119EF87" Ref="RN4"  Part="1"
-F 0 "RN4" H 2000 2705 59  0000 R BNN
+AR Path="/5F8FF86F/A119EF87" Ref="RN104"  Part="1"
+F 0 "RN104" H 2000 2705 59  0000 R BNN
 F 1 "DR1206-33R-4/8" H 2300 2580 59  0001 L BNN
 F 2 "EEZ DIB MCU r3B4:CAY16" H 2200 2700 50  0001 C CNN
@@
 AR Path="/5F88DC09/FDCEADBA97F649E4" Ref="RN6"  Part="3"
 AR Path="/5F8FF86F/FDCEADBA97F649E4" Ref="RN6"  Part="3"
-AR Path="/5F8FF86F/97F649E4" Ref="RN6"  Part="3"
-F 0 "RN6" H 2000 2605 59  0000 R BNN
+AR Path="/5F8FF86F/97F649E4" Ref="RN106"  Part="3"
+F 0 "RN106" H 2000 2605 59  0000 R BNN
 F 1 "DR1206-33R-4/8" H 2300 2480 59  0001 L BNN
 F 2 "EEZ DIB MCU r3B4:CAY16" H 2200 2600 50  0001 C CNN
@@
 AR Path="/5F88DC09/FDCEADBA97F649E0" Ref="RN6"  Part="2"
 AR Path="/5F8FF86F/FDCEADBA97F649E0" Ref="RN6"  Part="2"
-AR Path="/5F8FF86F/97F649E0" Ref="RN6"  Part="2"
-F 0 "RN6" H 2000 2505 59  0000 R BNN
+AR Path="/5F8FF86F/97F649E0" Ref="RN106"  Part="2"
+F 0 "RN106" H 2000 2505 59  0000 R BNN
 F 1 "DR1206-33R-4/8" H 2300 2380 59  0001 L BNN
 F 2 "EEZ DIB MCU r3B4:CAY16" H 2200 2500 50  0001 C CNN
@@
 AR Path="/5F88DC09/D4DDA4C0A119EF93" Ref="RN4"  Part="4"
 AR Path="/5F8FF86F/D4DDA4C0A119EF93" Ref="RN4"  Part="4"
-AR Path="/5F8FF86F/A119EF93" Ref="RN4"  Part="4"
-F 0 "RN4" H 2000 2005 59  0000 R BNN
+AR Path="/5F8FF86F/A119EF93" Ref="RN104"  Part="4"
+F 0 "RN104" H 2000 2005 59  0000 R BNN
 F 1 "DR1206-33R-4/8" H 2400 2005 59  0000 L BNN
 F 2 "EEZ DIB MCU r3B4:CAY16" H 2200 2000 50  0001 C CNN
@@
 	1    0    0    -1
 $EndComp
+$Comp
+L antena:CP_Small C166
+U 1 1 6143A283
+P 6600 4700
+F 0 "C166" H 6688 4746 50  0000 L CNN
+F 1 "10uF" H 6688 4655 50  0000 L CNN
+F 2 "Capacitor_Tantalum_SMD:CP_EIA-3216-10_Kemet-I" H 6600 4700 50  0001 C CNN
+F 3 "~" H 6600 4700 50  0001 C CNN
+	1    6600 4700
+	1    0    0    -1
+$EndComp
+Wire Wire Line
+	6600 4800 6600 5000
 $EndSCHEMATC
