File: Ethernet_PHY.sch (KiCad schematic (older format))
At the start: 44 parts, among them IC13 N.C., IC14 DP83848CVV_NOPB, X5 LMJTAB881243M-L

Commit message: More schematics cleanup
Changed lines of the file:
@@
 Text GLabel 7600 1200 0    10   BiDi ~ 0
 +3V3
-Wire Wire Line
-	1200 2600 2000 2600
-Text GLabel 1200 2600 2    50   BiDi ~ 0
+Text GLabel 1600 2600 0    50   BiDi ~ 0
 ETH_TX_EN
-Wire Wire Line
-	1200 2700 2000 2700
-Text GLabel 1200 2700 2    50   BiDi ~ 0
+Text GLabel 1600 2700 0    50   BiDi ~ 0
 ETH_RX_CLK
-Wire Wire Line
-	1200 2800 2000 2800
-Text GLabel 1200 2800 2    50   BiDi ~ 0
+Text GLabel 1600 2800 0    50   BiDi ~ 0
 ETH_RX_DV
-Wire Wire Line
-	2200 4100 1200 4100
-Text GLabel 1200 4100 2    50   BiDi ~ 0
+Text GLabel 1500 4100 0    50   BiDi ~ 0
 ETH_RXD0
-Wire Wire Line
-	1200 4200 2200 4200
-Text GLabel 1200 4200 2    50   BiDi ~ 0
+Text GLabel 1500 4200 0    50   BiDi ~ 0
 ETH_RXD1
-Wire Wire Line
-	1200 4300 2200 4300
-Text GLabel 1200 4300 2    50   BiDi ~ 0
+Text GLabel 1500 4300 0    50   BiDi ~ 0
 ETH_RXD2
-Wire Wire Line
-	1200 4400 2200 4400
-Text GLabel 1200 4400 2    50   BiDi ~ 0
+Text GLabel 1500 4400 0    50   BiDi ~ 0
 ETH_RXD3
-Wire Wire Line
-	1200 4600 2200 4600
-Text GLabel 1200 4600 2    50   BiDi ~ 0
+Text GLabel 1500 4600 0    50   BiDi ~ 0
 ETH_TXD0
-Wire Wire Line
-	1200 4700 2200 4700
-Text GLabel 1200 4700 2    50   BiDi ~ 0
+Text GLabel 1500 4700 0    50   BiDi ~ 0
 ETH_TXD1
-Wire Wire Line
-	1200 4800 2200 4800
-Text GLabel 1200 4800 2    50   BiDi ~ 0
+Text GLabel 1500 4800 0    50   BiDi ~ 0
 ETH_TXD2
-Wire Wire Line
-	1200 4900 2200 4900
-Text GLabel 1200 4900 2    50   BiDi ~ 0
+Text GLabel 1500 4900 0    50   BiDi ~ 0
 ETH_TXD3
-Wire Wire Line
-	1200 3800 3200 3800
-Text GLabel 1200 3800 2    50   BiDi ~ 0
+Text GLabel 1500 3800 0    50   BiDi ~ 0
 ~RESET
 Wire Wire Line
@@
 Connection ~ 2000 3700
 Wire Wire Line
-	1200 2300 3000 2300
-Wire Wire Line
 	3000 2300 3000 2500
 Wire Wire Line
 	3000 2500 3200 2500
-Text GLabel 1200 2300 2    50   BiDi ~ 0
+Text GLabel 1600 2300 0    50   BiDi ~ 0
 ETH_MDC
 Wire Wire Line
-	1200 2200 3100 2200
-Wire Wire Line
-	3100 2200 3100 2400
-Wire Wire Line
 	3100 2400 3200 2400
-Wire Wire Line
-	3100 2200 3100 2100
-Text GLabel 1200 2200 2    50   BiDi ~ 0
+Text GLabel 1600 2200 0    50   BiDi ~ 0
 ETH_MDIO
-Connection ~ 3100 2200
-Wire Wire Line
-	1200 2500 2000 2500
-Text GLabel 1200 2500 2    50   BiDi ~ 0
+Text GLabel 1600 2500 0    50   BiDi ~ 0
 ETH_TX_CLK
 Wire Wire Line
@@
 Wire Wire Line
 	9400 4800 7700 4800
-Wire Wire Line
-	1200 2000 2000 2000
-Text GLabel 1200 2000 2    50   BiDi ~ 0
+Text GLabel 1600 2000 0    50   BiDi ~ 0
 MCLK_25
 Wire Wire Line
@@
 	2900 2000 2900 2600
 Wire Wire Line
-	1200 3900 1900 3900
-Wire Wire Line
-	1900 3400 1900 3900
-Wire Wire Line
 	2200 3900 1900 3900
-Text GLabel 1200 3900 2    50   BiDi ~ 0
+Text GLabel 1500 3900 0    50   BiDi ~ 0
 ETH_CRS
-Connection ~ 1900 3900
 Wire Wire Line
 	3000 3500 3000 3400
@@
 Wire Wire Line
 	3200 3600 2600 3600
-Wire Wire Line
-	2200 3600 1200 3600
-Text GLabel 1200 3600 2    50   BiDi ~ 0
+Text GLabel 1500 3600 0    50   BiDi ~ 0
 ETH_COL
 Wire Wire Line
@@
 Wire Wire Line
 	2600 3900 3200 3900
-Wire Wire Line
-	1700 3700 1200 3700
-Text GLabel 1200 3700 2    50   BiDi ~ 0
+Text GLabel 1500 3700 0    50   BiDi ~ 0
 ETH_RX_ERR
 $Comp
@@
 Wire Wire Line
 	6600 4800 6600 5000
+Wire Wire Line
+	3100 2100 3100 2200
+Wire Wire Line
+	1600 2200 3100 2200
+Connection ~ 3100 2200
+Wire Wire Line
+	3100 2200 3100 2400
+Wire Wire Line
+	1600 2000 2000 2000
+Wire Wire Line
+	3000 2300 1600 2300
+Wire Wire Line
+	1600 2500 2000 2500
+Wire Wire Line
+	2000 2600 1600 2600
+Wire Wire Line
+	1600 2700 2000 2700
+Wire Wire Line
+	2000 2800 1600 2800
+Wire Wire Line
+	1900 3400 1900 3900
+Wire Wire Line
+	1500 3900 1900 3900
+Connection ~ 1900 3900
+Wire Wire Line
+	1500 3800 3200 3800
+Wire Wire Line
+	1500 3700 1700 3700
+Wire Wire Line
+	1500 3600 2200 3600
+Wire Wire Line
+	2200 4100 1500 4100
+Wire Wire Line
+	1500 4200 2200 4200
+Wire Wire Line
+	1500 4300 2200 4300
+Wire Wire Line
+	2200 4400 1500 4400
+Wire Wire Line
+	1500 4600 2200 4600
+Wire Wire Line
+	1500 4700 2200 4700
+Wire Wire Line
+	2200 4800 1500 4800
+Wire Wire Line
+	1500 4900 2200 4900
 $EndSCHEMATC

Commit message: Adding SPI from FPGA
Connections:
- net labels added: CLK_TO_ETH
- net labels removed: MCLK_25
Changed lines of the file:
@@
 Wire Wire Line
 	9400 4800 7700 4800
-Text GLabel 1600 2000 0    50   BiDi ~ 0
-MCLK_25
 Wire Wire Line
 	3200 2600 2900 2600
@@
 Wire Wire Line
 	1500 4900 2200 4900
+Text GLabel 1600 2000 0    60   Input ~ 0
+CLK_TO_ETH
 $EndSCHEMATC

Commit message: Routing FPGA to LCD
Parts:
- removed JP12: JP2-NOCUT, EEZ DIB MCU r3B4:JP2-NOCUT, symbol Ethernet_PHY-rescue:JP2-NOCUT-EEZ_DIB_MCU_r3B4-eagle-import
Connections:
- wire segments 228 -> 227
Changed lines of the file:
@@
 	2000 3000 2000 3300
-Wire Wire Line
-	3200 5000 2900 5000
-Wire Wire Line
-	2800 5000 2600 5000
 Wire Wire Line
 	2400 2500 2800 2500
@@
 $EndComp
 $Comp
-L Ethernet_PHY-rescue:JP2-NOCUT-EEZ_DIB_MCU_r3B4-eagle-import JP12
-U 1 1 01682B0F
-P 2800 5000
-AR Path="/BD05527201682B0F" Ref="JP12"  Part="1"
-AR Path="/5F88DC09/BD05527201682B0F" Ref="JP12"  Part="1"
-AR Path="/5F8FF86F/BD05527201682B0F" Ref="JP12"  Part="1"
-AR Path="/5F8FF86F/01682B0F" Ref="JP112"  Part="1"
-F 0 "JP112" H 2725 4900 59  0000 L BNN
-F 1 "JP2-NOCUT" H 2800 5000 50  0001 C CNN
-F 2 "EEZ DIB MCU r3B4:JP2-NOCUT" H 2800 5000 50  0001 C CNN
-F 3 "" H 2800 5000 50  0001 C CNN
-	1    2800 5000
-	1    0    0    -1
-$EndComp
-$Comp
 L Ethernet_PHY-rescue:+3V3-EEZ_DIB_MCU_r3B4-eagle-import #+3V334
 U 1 1 09D957BF
@@
 Text GLabel 1600 2000 0    60   Input ~ 0
 CLK_TO_ETH
+Wire Wire Line
+	2600 5000 3200 5000
 $EndSCHEMATC
