File: TFT_LCD_Audio_USB.sch (KiCad schematic (older format))
At the start: 35 parts, among them IC10 TPS61169DCKR, IC11 TPD4E001DRLR, IC12 TSC2007IPW, IC9 TPS2051BDBVR, J2 67803-8020, Q1 N.C., Q2 2N7002

Commit message: Adding default parts
Parts:
- C50, C56: footprint EEZ DIB MCU r3B4:C1206 -> Capacitor_SMD:C_1206_3216Metric
- C51, C53, C58: footprint EEZ DIB MCU r3B4:C0805 -> Capacitor_SMD:C_0805_2012Metric
- C52: footprint EEZ DIB MCU r3B4:EC1206 -> Capacitor_SMD:C_1206_3216Metric
- C54: footprint EEZ DIB MCU r3B4:C1812 -> Capacitor_SMD:C_1812_4532Metric
- C55, C57: footprint EEZ DIB MCU r3B4:C0603 -> Capacitor_SMD:C_0603_1608Metric
- R24, R25, R26, R27, R28, R29, R30, R31, R32, R33: footprint EEZ DIB MCU r3B4:R0805 -> Resistor_SMD:R_0805_2012Metric
Changed lines of the file:
@@
 F 0 "R126" V 3291 2150 59  0000 L BNN
 F 1 "10R" V 3380 2150 59  0000 L BNN
-F 2 "EEZ DIB MCU r3B4:R0805" H 3300 2100 50  0001 C CNN
+F 2 "Resistor_SMD:R_0805_2012Metric" H 3300 2100 50  0001 C CNN
 F 3 "" H 3300 2100 50  0001 C CNN
 	1    3300 2100
@@
 F 0 "C150" H 1515 1410 59  0000 R TNN
 F 1 "4u7" H 1515 1335 59  0000 R TNN
-F 2 "EEZ DIB MCU r3B4:C1206" H 1600 1400 50  0001 C CNN
+F 2 "Capacitor_SMD:C_1206_3216Metric" H 1600 1400 50  0001 C CNN
 F 3 "" H 1600 1400 50  0001 C CNN
 	1    1600 1400
@@
 F 0 "C151" H 3415 1435 59  0000 R TNN
 F 1 "1u" H 3415 1335 59  0000 R TNN
-F 2 "EEZ DIB MCU r3B4:C0805" H 3500 1400 50  0001 C CNN
+F 2 "Capacitor_SMD:C_0805_2012Metric" H 3500 1400 50  0001 C CNN
 F 3 "" H 3500 1400 50  0001 C CNN
 	1    3500 1400
@@
 F 0 "C157" H 5710 5640 59  0000 L BNN
 F 1 "100n" H 5710 5860 59  0000 L TNN
-F 2 "EEZ DIB MCU r3B4:C0603" H 5700 5800 50  0001 C CNN
+F 2 "Capacitor_SMD:C_0603_1608Metric" H 5700 5800 50  0001 C CNN
 F 3 "" H 5700 5800 50  0001 C CNN
 	1    5700 5800
@@
 F 0 "C158" H 5990 5710 59  0000 R TNN
 F 1 "1u" H 5990 5860 59  0000 R TNN
-F 2 "EEZ DIB MCU r3B4:C0805" H 6000 5800 50  0001 C CNN
+F 2 "Capacitor_SMD:C_0805_2012Metric" H 6000 5800 50  0001 C CNN
 F 3 "" H 6000 5800 50  0001 C CNN
 	1    6000 5800
@@
 F 0 "R133" H 3700 3640 59  0000 R TNN
 F 1 "10K" H 3700 3815 59  0000 R TNN
-F 2 "EEZ DIB MCU r3B4:R0805" H 3600 3700 50  0001 C CNN
+F 2 "Resistor_SMD:R_0805_2012Metric" H 3600 3700 50  0001 C CNN
 F 3 "" H 3600 3700 50  0001 C CNN
 	1    3600 3700
@@
 F 0 "R124" V 1891 1450 59  0000 R BNN
 F 1 "10R" V 1980 1450 59  0000 R BNN
-F 2 "EEZ DIB MCU r3B4:R0805" H 1900 1500 50  0001 C CNN
+F 2 "Resistor_SMD:R_0805_2012Metric" H 1900 1500 50  0001 C CNN
 F 3 "" H 1900 1500 50  0001 C CNN
 	1    1900 1500
@@
 F 0 "C153" H 4215 2365 59  0000 R BNN
 F 1 "2u2" H 4215 2290 59  0000 R BNN
-F 2 "EEZ DIB MCU r3B4:C0805" H 4300 2400 50  0001 C CNN
+F 2 "Capacitor_SMD:C_0805_2012Metric" H 4300 2400 50  0001 C CNN
 F 3 "" H 4300 2400 50  0001 C CNN
 	1    4300 2400
@@
 F 0 "C156" V 7885 4685 59  0000 L BNN
 F 1 "4u7" V 7785 4685 59  0000 L BNN
-F 2 "EEZ DIB MCU r3B4:C1206" H 7800 4700 50  0001 C CNN
+F 2 "Capacitor_SMD:C_1206_3216Metric" H 7800 4700 50  0001 C CNN
 F 3 "" H 7800 4700 50  0001 C CNN
 	1    7800 4700
@@
 F 0 "R130" H 8900 2710 59  0000 R BNN
 F 1 "22R" H 8475 2710 59  0000 R BNN
-F 2 "EEZ DIB MCU r3B4:R0805" H 8600 2700 50  0001 C CNN
+F 2 "Resistor_SMD:R_0805_2012Metric" H 8600 2700 50  0001 C CNN
 F 3 "" H 8600 2700 50  0001 C CNN
 	1    8600 2700
@@
 F 0 "R131" H 8900 2810 59  0000 R BNN
 F 1 "22R" H 8475 2810 59  0000 R BNN
-F 2 "EEZ DIB MCU r3B4:R0805" H 8600 2800 50  0001 C CNN
+F 2 "Resistor_SMD:R_0805_2012Metric" H 8600 2800 50  0001 C CNN
 F 3 "" H 8600 2800 50  0001 C CNN
 	1    8600 2800
@@
 F 0 "R127" V 7791 1950 59  0000 L BNN
 F 1 "10K" V 7705 1950 59  0000 L BNN
-F 2 "EEZ DIB MCU r3B4:R0805" H 7700 1900 50  0001 C CNN
+F 2 "Resistor_SMD:R_0805_2012Metric" H 7700 1900 50  0001 C CNN
 F 3 "" H 7700 1900 50  0001 C CNN
 	1    7700 1900
@@
 F 0 "C155" H 8285 3535 59  0000 L TNN
 F 1 "100n" H 8285 3610 59  0000 L TNN
-F 2 "EEZ DIB MCU r3B4:C0603" H 8200 3600 50  0001 C CNN
+F 2 "Capacitor_SMD:C_0603_1608Metric" H 8200 3600 50  0001 C CNN
 F 3 "" H 8200 3600 50  0001 C CNN
 	1    8200 3600
@@
 F 0 "C152" H 9505 1625 59  0000 R TNN
 F 1 "4u7" H 9505 1540 59  0000 R TNN
-F 2 "EEZ DIB MCU r3B4:EC1206" H 9600 1600 50  0001 C CNN
+F 2 "Capacitor_SMD:C_1206_3216Metric" H 9600 1600 50  0001 C CNN
 F 3 "" H 9600 1600 50  0001 C CNN
 	1    9600 1600
@@
 F 0 "R128" V 10291 2350 59  0000 L BNN
 F 1 "N.C." V 10205 2350 59  0000 L BNN
-F 2 "EEZ DIB MCU r3B4:R0805" H 10200 2300 50  0001 C CNN
+F 2 "Resistor_SMD:R_0805_2012Metric" H 10200 2300 50  0001 C CNN
 F 3 "" H 10200 2300 50  0001 C CNN
 	1    10200 2300
@@
 F 0 "R125" V 10666 1650 59  0000 L BNN
 F 1 "N.C." V 10580 1650 59  0000 L BNN
-F 2 "EEZ DIB MCU r3B4:R0805" H 10600 1600 50  0001 C CNN
+F 2 "Resistor_SMD:R_0805_2012Metric" H 10600 1600 50  0001 C CNN
 F 3 "" H 10600 1600 50  0001 C CNN
 	1    10600 1600
@@
 F 0 "C154" V 10085 3310 59  0000 L BNN
 F 1 "4n7/1kV" V 10185 3310 59  0000 L BNN
-F 2 "EEZ DIB MCU r3B4:C1812" H 10100 3300 50  0001 C CNN
+F 2 "Capacitor_SMD:C_1812_4532Metric" H 10100 3300 50  0001 C CNN
 F 3 "" H 10100 3300 50  0001 C CNN
 	1    10100 3300
@@
 F 0 "R129" H 7975 2735 59  0000 R BNN
 F 1 "4K7" H 7975 2660 59  0000 R BNN
-F 2 "EEZ DIB MCU r3B4:R0805" H 7900 2600 50  0001 C CNN
+F 2 "Resistor_SMD:R_0805_2012Metric" H 7900 2600 50  0001 C CNN
 F 3 "" H 7900 2600 50  0001 C CNN
 	1    7900 2600
@@
 F 0 "R132" V 7610 3225 59  0000 L TNN
 F 1 "10K" V 7710 3250 59  0000 L TNN
-F 2 "EEZ DIB MCU r3B4:R0805" H 7700 3200 50  0001 C CNN
+F 2 "Resistor_SMD:R_0805_2012Metric" H 7700 3200 50  0001 C CNN
 F 3 "" H 7700 3200 50  0001 C CNN
 	1    7700 3200

Commit message: Adding TO FROM FPGA lines
Connections:
- net labels added: LTDC_FROM_FPGA_B3, LTDC_FROM_FPGA_B4, LTDC_FROM_FPGA_B5, LTDC_FROM_FPGA_B6, LTDC_FROM_FPGA_B7, LTDC_FROM_FPGA_CLK, LTDC_FROM_FPGA_DE, LTDC_FROM_FPGA_G2, LTDC_FROM_FPGA_G3, LTDC_FROM_FPGA_G4, LTDC_FROM_FPGA_G5, LTDC_FROM_FPGA_G6, LTDC_FROM_FPGA_G7, LTDC_FROM_FPGA_HSYNC, LTDC_FROM_FPGA_R3, LTDC_FROM_FPGA_R4, LTDC_FROM_FPGA_R5, LTDC_FROM_FPGA_R6, LTDC_FROM_FPGA_R7, LTDC_FROM_FPGA_VSYNC
- net labels removed: LTDC_B3, LTDC_B4, LTDC_B5, LTDC_B6, LTDC_B7, LTDC_CLK, LTDC_DE, LTDC_G2, LTDC_G3, LTDC_G4, LTDC_G5, LTDC_G6, LTDC_G7, LTDC_HSYNC, LTDC_R3, LTDC_R4, LTDC_R5, LTDC_R6, LTDC_R7, LTDC_VSYNC
Changed lines of the file:
@@
 	4700 3100 3100 3100
 Text GLabel 3100 3100 2    50   BiDi ~ 0
-LTDC_CLK
+LTDC_FROM_FPGA_CLK
 Wire Wire Line
 	4700 3300 3100 3300
 Text GLabel 3100 3300 2    50   BiDi ~ 0
-LTDC_HSYNC
+LTDC_FROM_FPGA_HSYNC
 Wire Wire Line
 	4700 3400 3100 3400
 Text GLabel 3100 3400 2    50   BiDi ~ 0
-LTDC_VSYNC
+LTDC_FROM_FPGA_VSYNC
 Wire Wire Line
 	4700 3500 3100 3500
 Text GLabel 3100 3500 2    50   BiDi ~ 0
-LTDC_DE
+LTDC_FROM_FPGA_DE
 Wire Wire Line
 	4700 3200 3900 3200
@@
 	5700 4200 6200 4200
 Text GLabel 6200 4200 0    50   BiDi ~ 0
-LTDC_B7
+LTDC_FROM_FPGA_B7
 Wire Wire Line
 	5700 4100 6200 4100
 Text GLabel 6200 4100 0    50   BiDi ~ 0
-LTDC_B6
+LTDC_FROM_FPGA_B6
 Wire Wire Line
 	5700 4000 6200 4000
 Text GLabel 6200 4000 0    50   BiDi ~ 0
-LTDC_B5
+LTDC_FROM_FPGA_B5
 Wire Wire Line
 	5700 3900 6200 3900
 Text GLabel 6200 3900 0    50   BiDi ~ 0
-LTDC_B4
+LTDC_FROM_FPGA_B4
 Wire Wire Line
 	5700 3800 6200 3800
 Text GLabel 6200 3800 0    50   BiDi ~ 0
-LTDC_B3
+LTDC_FROM_FPGA_B3
 Wire Wire Line
 	5700 3400 6200 3400
 Text GLabel 6200 3400 0    50   BiDi ~ 0
-LTDC_G7
+LTDC_FROM_FPGA_G7
 Wire Wire Line
 	5700 2600 6200 2600
 Text GLabel 6200 2600 0    50   BiDi ~ 0
-LTDC_R7
+LTDC_FROM_FPGA_R7
 Wire Wire Line
 	5700 2500 6200 2500
 Text GLabel 6200 2500 0    50   BiDi ~ 0
-LTDC_R6
+LTDC_FROM_FPGA_R6
 Wire Wire Line
 	5700 2400 6200 2400
 Text GLabel 6200 2400 0    50   BiDi ~ 0
-LTDC_R5
+LTDC_FROM_FPGA_R5
 Wire Wire Line
 	5700 2300 6200 2300
 Text GLabel 6200 2300 0    50   BiDi ~ 0
-LTDC_R4
+LTDC_FROM_FPGA_R4
 Wire Wire Line
 	5700 2200 6200 2200
 Text GLabel 6200 2200 0    50   BiDi ~ 0
-LTDC_R3
+LTDC_FROM_FPGA_R3
 Wire Wire Line
 	5500 6400 6100 6400
@@
 	5700 2900 6200 2900
 Text GLabel 6200 2900 0    50   BiDi ~ 0
-LTDC_G2
+LTDC_FROM_FPGA_G2
 Wire Wire Line
 	5700 3000 6200 3000
 Text GLabel 6150 3000 0    50   BiDi ~ 0
-LTDC_G3
+LTDC_FROM_FPGA_G3
 Wire Wire Line
 	5700 3100 6200 3100
 Text GLabel 6200 3100 0    50   BiDi ~ 0
-LTDC_G4
+LTDC_FROM_FPGA_G4
 Wire Wire Line
 	5700 3200 6200 3200
 Text GLabel 6200 3200 0    50   BiDi ~ 0
-LTDC_G5
+LTDC_FROM_FPGA_G5
 Wire Wire Line
 	5700 3300 6200 3300
 Text GLabel 6200 3300 0    50   BiDi ~ 0
-LTDC_G6
+LTDC_FROM_FPGA_G6
 Wire Wire Line
 	7800 5600 7300 5600

Commit message: Rewiering LCD OUT to bottom left
Parts:
- removed C52: 4u7, Capacitor_SMD:C_1206_3216Metric, symbol TFT_LCD_Audio_USB-rescue:ECAP1206-EEZ_DIB_MCU_r3B4-eagle-import
- added C152: 4u7, Capacitor_Tantalum_SMD:CP_EIA-3216-10_Kemet-I, symbol antena:CP_Small
- R24, R25, R26, R27, R28, R32, R33: footprint Resistor_SMD:R_0805_2012Metric -> Resistor_SMD:R_0603_1608Metric
Changed lines of the file:
@@
 Text GLabel 8300 3700 0    10   BiDi ~ 0
 GND
-Wire Wire Line
-	9600 1900 9600 1800
 Text GLabel 9600 1900 0    10   BiDi ~ 0
 GND
@@
 Wire Wire Line
 	9400 1400 9600 1400
-Wire Wire Line
-	9600 1400 9600 1500
 Wire Wire Line
 	10200 2500 10200 2600
@@
 F 0 "R126" V 3291 2150 59  0000 L BNN
 F 1 "10R" V 3380 2150 59  0000 L BNN
-F 2 "Resistor_SMD:R_0805_2012Metric" H 3300 2100 50  0001 C CNN
+F 2 "Resistor_SMD:R_0603_1608Metric" H 3300 2100 50  0001 C CNN
 F 3 "" H 3300 2100 50  0001 C CNN
 	1    3300 2100
@@
 F 0 "R133" H 3700 3640 59  0000 R TNN
 F 1 "10K" H 3700 3815 59  0000 R TNN
-F 2 "Resistor_SMD:R_0805_2012Metric" H 3600 3700 50  0001 C CNN
+F 2 "Resistor_SMD:R_0603_1608Metric" H 3600 3700 50  0001 C CNN
 F 3 "" H 3600 3700 50  0001 C CNN
 	1    3600 3700
@@
 F 0 "R124" V 1891 1450 59  0000 R BNN
 F 1 "10R" V 1980 1450 59  0000 R BNN
-F 2 "Resistor_SMD:R_0805_2012Metric" H 1900 1500 50  0001 C CNN
+F 2 "Resistor_SMD:R_0603_1608Metric" H 1900 1500 50  0001 C CNN
 F 3 "" H 1900 1500 50  0001 C CNN
 	1    1900 1500
@@
 F 0 "R127" V 7791 1950 59  0000 L BNN
 F 1 "10K" V 7705 1950 59  0000 L BNN
-F 2 "Resistor_SMD:R_0805_2012Metric" H 7700 1900 50  0001 C CNN
+F 2 "Resistor_SMD:R_0603_1608Metric" H 7700 1900 50  0001 C CNN
 F 3 "" H 7700 1900 50  0001 C CNN
 	1    7700 1900
@@
 $EndComp
 $Comp
-L TFT_LCD_Audio_USB-rescue:ECAP1206-EEZ_DIB_MCU_r3B4-eagle-import C52
-U 1 1 9BA5F96A
-P 9600 1600
-AR Path="/BBA627E59BA5F96A" Ref="C52"  Part="1"
-AR Path="/5F88D857/BBA627E59BA5F96A" Ref="C52"  Part="1"
-AR Path="/5F8FBDC2/9BA5F96A" Ref="C152"  Part="1"
-F 0 "C152" H 9505 1625 59  0000 R TNN
-F 1 "4u7" H 9505 1540 59  0000 R TNN
-F 2 "Capacitor_SMD:C_1206_3216Metric" H 9600 1600 50  0001 C CNN
-F 3 "" H 9600 1600 50  0001 C CNN
-	1    9600 1600
-	-1   0    0    -1
-$EndComp
-$Comp
 L TFT_LCD_Audio_USB-rescue:GND-EEZ_DIB_MCU_r3B4-eagle-import #SUPPLY49
 U 1 1 8FADADE5
@@
 F 0 "R128" V 10291 2350 59  0000 L BNN
 F 1 "N.C." V 10205 2350 59  0000 L BNN
-F 2 "Resistor_SMD:R_0805_2012Metric" H 10200 2300 50  0001 C CNN
+F 2 "Resistor_SMD:R_0603_1608Metric" H 10200 2300 50  0001 C CNN
 F 3 "" H 10200 2300 50  0001 C CNN
 	1    10200 2300
@@
 F 0 "R125" V 10666 1650 59  0000 L BNN
 F 1 "N.C." V 10580 1650 59  0000 L BNN
-F 2 "Resistor_SMD:R_0805_2012Metric" H 10600 1600 50  0001 C CNN
+F 2 "Resistor_SMD:R_0603_1608Metric" H 10600 1600 50  0001 C CNN
 F 3 "" H 10600 1600 50  0001 C CNN
 	1    10600 1600
@@
 F 0 "R132" V 7610 3225 59  0000 L TNN
 F 1 "10K" V 7710 3250 59  0000 L TNN
-F 2 "Resistor_SMD:R_0805_2012Metric" H 7700 3200 50  0001 C CNN
+F 2 "Resistor_SMD:R_0603_1608Metric" H 7700 3200 50  0001 C CNN
 F 3 "" H 7700 3200 50  0001 C CNN
 	1    7700 3200
@@
 Wire Notes Line
 	6900 900  6900 6500
+$Comp
+L antena:CP_Small C152
+U 1 1 6149B513
+P 9600 1650
+F 0 "C152" H 9688 1696 50  0000 L CNN
+F 1 "4u7" H 9688 1605 50  0000 L CNN
+F 2 "Capacitor_Tantalum_SMD:CP_EIA-3216-10_Kemet-I" H 9600 1650 50  0001 C CNN
+F 3 "~" H 9600 1650 50  0001 C CNN
+	1    9600 1650
+	1    0    0    -1
+$EndComp
+Wire Wire Line
+	9600 1400 9600 1550
+Wire Wire Line
+	9600 1750 9600 1900
 Wire Bus Line
 	6300 2000 6300 4100

Commit message: LCD connector cleanup
Connections:
- net labels removed: LTDC_R[2..7],LTDC_G[2..7],LTDC_B[2..7]
Changed lines of the file:
@@
 Comment4 ""
 $EndDescr
-Wire Bus Line
-	6300 2000 6400 1900
-Wire Bus Line
-	6400 1900 6700 1900
-Text Label 6300 3050 1    50   ~ 0
-LTDC_R[2..7],LTDC_G[2..7],LTDC_B[2..7]
 Wire Wire Line
 	10500 3500 10500 3300
@@
 	3000 1200 3200 1200
 Connection ~ 3000 1200
-Wire Wire Line
-	4700 3100 3100 3100
-Text GLabel 3100 3100 2    50   BiDi ~ 0
+Text GLabel 3800 3100 0    50   BiDi ~ 0
 LTDC_FROM_FPGA_CLK
-Wire Wire Line
-	4700 3300 3100 3300
-Text GLabel 3100 3300 2    50   BiDi ~ 0
+Text GLabel 3800 3300 0    50   BiDi ~ 0
 LTDC_FROM_FPGA_HSYNC
-Wire Wire Line
-	4700 3400 3100 3400
-Text GLabel 3100 3400 2    50   BiDi ~ 0
+Text GLabel 3800 3400 0    50   BiDi ~ 0
 LTDC_FROM_FPGA_VSYNC
-Wire Wire Line
-	4700 3500 3100 3500
-Text GLabel 3100 3500 2    50   BiDi ~ 0
+Text GLabel 3800 3500 0    50   BiDi ~ 0
 LTDC_FROM_FPGA_DE
 Wire Wire Line
@@
 Text Label 4300 5900 2    50   ~ 0
 YU
-Wire Wire Line
-	5700 4200 6200 4200
-Text GLabel 6200 4200 0    50   BiDi ~ 0
+Text GLabel 5850 4200 2    50   BiDi ~ 0
 LTDC_FROM_FPGA_B7
-Wire Wire Line
-	5700 4100 6200 4100
-Text GLabel 6200 4100 0    50   BiDi ~ 0
+Text GLabel 5850 4100 2    50   BiDi ~ 0
 LTDC_FROM_FPGA_B6
-Wire Wire Line
-	5700 4000 6200 4000
-Text GLabel 6200 4000 0    50   BiDi ~ 0
+Text GLabel 5850 4000 2    50   BiDi ~ 0
 LTDC_FROM_FPGA_B5
-Wire Wire Line
-	5700 3900 6200 3900
-Text GLabel 6200 3900 0    50   BiDi ~ 0
+Text GLabel 5850 3900 2    50   BiDi ~ 0
 LTDC_FROM_FPGA_B4
-Wire Wire Line
-	5700 3800 6200 3800
-Text GLabel 6200 3800 0    50   BiDi ~ 0
+Text GLabel 5850 3800 2    50   BiDi ~ 0
 LTDC_FROM_FPGA_B3
-Wire Wire Line
-	5700 3400 6200 3400
-Text GLabel 6200 3400 0    50   BiDi ~ 0
+Text GLabel 5850 3400 2    50   BiDi ~ 0
 LTDC_FROM_FPGA_G7
-Wire Wire Line
-	5700 2600 6200 2600
-Text GLabel 6200 2600 0    50   BiDi ~ 0
+Text GLabel 5850 2600 2    50   BiDi ~ 0
 LTDC_FROM_FPGA_R7
-Wire Wire Line
-	5700 2500 6200 2500
-Text GLabel 6200 2500 0    50   BiDi ~ 0
+Text GLabel 5850 2500 2    50   BiDi ~ 0
 LTDC_FROM_FPGA_R6
-Wire Wire Line
-	5700 2400 6200 2400
-Text GLabel 6200 2400 0    50   BiDi ~ 0
+Text GLabel 5850 2400 2    50   BiDi ~ 0
 LTDC_FROM_FPGA_R5
-Wire Wire Line
-	5700 2300 6200 2300
-Text GLabel 6200 2300 0    50   BiDi ~ 0
+Text GLabel 5850 2300 2    50   BiDi ~ 0
 LTDC_FROM_FPGA_R4
-Wire Wire Line
-	5700 2200 6200 2200
-Text GLabel 6200 2200 0    50   BiDi ~ 0
+Text GLabel 5850 2200 2    50   BiDi ~ 0
 LTDC_FROM_FPGA_R3
 Wire Wire Line
@@
 Text GLabel 6100 6400 0    50   BiDi ~ 0
 IRQ_TOUCH
-Wire Wire Line
-	5700 2900 6200 2900
-Text GLabel 6200 2900 0    50   BiDi ~ 0
+Text GLabel 5850 2900 2    50   BiDi ~ 0
 LTDC_FROM_FPGA_G2
-Wire Wire Line
-	5700 3000 6200 3000
-Text GLabel 6150 3000 0    50   BiDi ~ 0
+Text GLabel 5850 3000 2    50   BiDi ~ 0
 LTDC_FROM_FPGA_G3
-Wire Wire Line
-	5700 3100 6200 3100
-Text GLabel 6200 3100 0    50   BiDi ~ 0
+Text GLabel 5850 3100 2    50   BiDi ~ 0
 LTDC_FROM_FPGA_G4
-Wire Wire Line
-	5700 3200 6200 3200
-Text GLabel 6200 3200 0    50   BiDi ~ 0
+Text GLabel 5850 3200 2    50   BiDi ~ 0
 LTDC_FROM_FPGA_G5
-Wire Wire Line
-	5700 3300 6200 3300
-Text GLabel 6200 3300 0    50   BiDi ~ 0
+Text GLabel 5850 3300 2    50   BiDi ~ 0
 LTDC_FROM_FPGA_G6
 Wire Wire Line
@@
 DAC_OUT1
 Wire Wire Line
-	7000 2600 7700 2600
-Wire Wire Line
 	7700 3000 7700 2600
-Text GLabel 7000 2600 2    50   BiDi ~ 0
+Text GLabel 7650 2600 0    50   BiDi ~ 0
 USB_OTG_FS_VBUS
-Connection ~ 7700 2600
-Wire Wire Line
-	7000 2900 9600 2900
 Wire Wire Line
 	9600 2900 10600 2900
@@
 Wire Wire Line
 	9600 3600 9600 2900
-Text GLabel 7000 2900 2    50   BiDi ~ 0
+Text GLabel 7650 2900 0    50   BiDi ~ 0
 USB_OTG_FS_ID
-Connection ~ 9600 2900
-Wire Wire Line
-	8400 2700 7000 2700
-Text GLabel 7000 2700 2    50   BiDi ~ 0
+Text GLabel 7650 2700 0    50   BiDi ~ 0
 USB_OTG_FS_D_N
-Wire Wire Line
-	7000 2800 8400 2800
-Text GLabel 7000 2800 2    50   BiDi ~ 0
+Text GLabel 7650 2800 0    50   BiDi ~ 0
 USB_OTG_FS_D_P
 Wire Wire Line
@@
 Text GLabel 1600 1300 0    10   BiDi ~ 0
 +5V
-Wire Wire Line
-	8100 1600 7000 1600
-Text GLabel 7000 1600 2    50   BiDi ~ 0
+Text GLabel 7650 1600 0    50   BiDi ~ 0
 ~USB_OTG_FS_OC
 Wire Wire Line
 	8100 1500 7700 1500
-Wire Wire Line
-	7700 1500 7000 1500
-Wire Wire Line
-	7700 1700 7700 1500
-Text GLabel 7000 1500 2    50   BiDi ~ 0
+Text GLabel 7650 1500 0    50   BiDi ~ 0
 USB_OTG_FS_PSO
-Connection ~ 7700 1500
 Wire Wire Line
 	10400 2000 10200 2000
@@
 Connection ~ 8200 2600
 Connection ~ 8200 3400
-Entry Wire Line
-	6200 4200 6300 4100
-Entry Wire Line
-	6200 4100 6300 4000
-Entry Wire Line
-	6200 4000 6300 3900
-Entry Wire Line
-	6200 3900 6300 3800
-Entry Wire Line
-	6200 3800 6300 3700
-Entry Wire Line
-	6200 3400 6300 3300
-Entry Wire Line
-	6200 2600 6300 2500
-Entry Wire Line
-	6200 2500 6300 2400
-Entry Wire Line
-	6200 2400 6300 2300
-Entry Wire Line
-	6200 2300 6300 2200
-Entry Wire Line
-	6200 2200 6300 2100
-Entry Wire Line
-	6200 2900 6300 2800
-Entry Wire Line
-	6200 3000 6300 2900
-Entry Wire Line
-	6200 3100 6300 3000
-Entry Wire Line
-	6200 3200 6300 3100
-Entry Wire Line
-	6200 3300 6300 3200
 $Comp
 L TFT_LCD_Audio_USB-rescue:DINA4_L-EEZ_DIB_MCU_r3B4-eagle-import #FRAME4
@@
 Wire Wire Line
 	9600 1750 9600 1900
-Wire Bus Line
-	6300 2000 6300 4100
+Wire Wire Line
+	7650 2600 7700 2600
+Connection ~ 7700 2600
+Wire Wire Line
+	8400 2700 7650 2700
+Wire Wire Line
+	8400 2800 7650 2800
+Wire Wire Line
+	7650 2900 9600 2900
+Connection ~ 9600 2900
+Wire Wire Line
+	7700 1700 7700 1500
+Wire Wire Line
+	7650 1600 8100 1600
+Wire Wire Line
+	7650 1500 7700 1500
+Connection ~ 7700 1500
+Wire Wire Line
+	3800 3100 4700 3100
+Wire Wire Line
+	4700 3300 3800 3300
+Wire Wire Line
+	3800 3400 4700 3400
+Wire Wire Line
+	4700 3500 3800 3500
+Wire Wire Line
+	5850 2200 5700 2200
+Wire Wire Line
+	5700 2300 5850 2300
+Wire Wire Line
+	5850 2400 5700 2400
+Wire Wire Line
+	5700 2500 5850 2500
+Wire Wire Line
+	5850 2600 5700 2600
+Wire Wire Line
+	5700 2900 5850 2900
+Wire Wire Line
+	5850 3000 5700 3000
+Wire Wire Line
+	5700 3100 5850 3100
+Wire Wire Line
+	5850 3200 5700 3200
+Wire Wire Line
+	5700 3300 5850 3300
+Wire Wire Line
+	5850 3400 5700 3400
+Wire Wire Line
+	5850 3800 5700 3800
+Wire Wire Line
+	5700 3900 5850 3900
+Wire Wire Line
+	5850 4000 5700 4000
+Wire Wire Line
+	5850 4100 5700 4100
+Wire Wire Line
+	5700 4200 5850 4200
 $EndSCHEMATC
