File: TFT_LCD_Audio_USB.sch (KiCad schematic (older format))
At the start: 35 parts, among them IC10 TPS61169DCKR, IC11 TPD4E001DRLR, IC12 TSC2007IPW, IC9 TPS2051BDBVR, J2 67803-8020, Q1 N.C., Q2 2N7002

Commit message: Routing long signals
Parts:
- removed SH1: SHORTNOHOLE, EEZ DIB MCU r3B4:SHORT_NOHOLE, symbol TFT_LCD_Audio_USB-rescue:SHORTNOHOLE-EEZ_DIB_MCU_r3B4-eagle-import
Changed lines of the file:
@@
 Wire Wire Line
 	8000 4700 8000 4600
-Wire Wire Line
-	8000 4800 8000 4700
 Connection ~ 8000 4700
 Text GLabel 8000 4700 0    10   BiDi ~ 0
@@
 	1    10100 3300
 	0    -1   1    0
-$EndComp
-$Comp
-L TFT_LCD_Audio_USB-rescue:SHORTNOHOLE-EEZ_DIB_MCU_r3B4-eagle-import SH1
-U 1 1 EC26DEFE
-P 8000 4900
-AR Path="/990531BEC26DEFE" Ref="SH1"  Part="1"
-AR Path="/5F88D857/990531BEC26DEFE" Ref="SH1"  Part="1"
-AR Path="/5F8FBDC2/EC26DEFE" Ref="SH101"  Part="1"
-F 0 "SH101" H 7913 4950 59  0000 L BNN
-F 1 "SHORTNOHOLE" H 8000 4900 50  0001 C CNN
-F 2 "EEZ DIB MCU r3B4:SHORT_NOHOLE" H 8000 4900 50  0001 C CNN
-F 3 "" H 8000 4900 50  0001 C CNN
-	1    8000 4900
-	0    1    -1   0
 $EndComp
 $Comp
@@
 Wire Wire Line
 	5700 4200 5850 4200
+Wire Wire Line
+	8000 4700 8000 5000
 $EndSCHEMATC

Commit message: V0.1
Parts:
- added J2: USB_OTG, usb_otg:USB-MICRO-B-FCI-10118192-0001LF-small-pads, symbol Connector:USB_OTG
Connections:
- wire segments 159 -> 180
Changed lines of the file:
@@
 EESchema Schematic File Version 4
-LIBS:ulx3s-cache
-EELAYER 29 0
+EELAYER 30 0
 EELAYER END
 $Descr User 12118 8710
@@
 USB_OTG_FS_VBUS
 Wire Wire Line
-	9600 2900 10600 2900
+	9600 2900 10350 2900
 Wire Wire Line
 	9300 3600 9600 3600
@@
 	8800 2800 9500 2800
 Wire Wire Line
-	9500 2800 10600 2800
+	9500 2800 10550 2800
 Wire Wire Line
 	9300 3500 9500 3500
@@
 	8800 2700 9400 2700
 Wire Wire Line
-	9400 2700 10600 2700
+	9400 2700 10500 2700
 Wire Wire Line
 	9300 3400 9400 3400
@@
 	8200 2600 9400 2600
 Wire Wire Line
-	9400 2600 10200 2600
+	9400 2600 9700 2600
 Wire Wire Line
 	9100 1400 9400 1400
@@
 L TFT_LCD_Audio_USB-rescue:GND-EEZ_DIB_MCU_r3B4-eagle-import #SUPPLY51
 U 1 1 294709DD
-P 10600 2300
+P 11300 2200
 AR Path="/6C78D67F294709DD" Ref="#SUPPLY51"  Part="1"
 AR Path="/5F88D857/6C78D67F294709DD" Ref="#SUPPLY051"  Part="1"
 AR Path="/5F8FBDC2/294709DD" Ref="#SUPPLY051"  Part="1"
-F 0 "#SUPPLY051" H 10600 2300 50  0001 C CNN
-F 1 "PGND" H 10665 2350 59  0000 L TNN
-F 2 "" H 10600 2300 50  0001 C CNN
-F 3 "" H 10600 2300 50  0001 C CNN
-	1    10600 2300
-	1    0    0    -1
+F 0 "#SUPPLY051" H 11300 2200 50  0001 C CNN
+F 1 "PGND" H 11365 2250 59  0000 L TNN
+F 2 "" H 11300 2200 50  0001 C CNN
+F 3 "" H 11300 2200 50  0001 C CNN
+	1    11300 2200
+	0    -1   -1   0
 $EndComp
 $Comp
@@
 Wire Wire Line
 	8000 4700 8000 5000
+$Comp
+L Connector:USB_OTG J2
+U 1 1 5FA161B6
+P 11950 2800
+F 0 "J2" H 11720 2697 50  0000 R CNN
+F 1 "USB_OTG" H 11720 2788 50  0000 R CNN
+F 2 "usb_otg:USB-MICRO-B-FCI-10118192-0001LF-small-pads" H 12100 2750 50  0001 C CNN
+F 3 " ~" H 12100 2750 50  0001 C CNN
+	1    11950 2800
+	-1   0    0    1
+$EndComp
+$Comp
+L TFT_LCD_Audio_USB-rescue:PE-EEZ_DIB_MCU_r3B4-eagle-import #PE?
+U 1 1 5FA1E6B6
+P 12050 2300
+AR Path="/6C68606E5FA1E6B6" Ref="#PE?"  Part="1"
+AR Path="/5F88D857/6C68606E5FA1E6B6" Ref="#PE?"  Part="1"
+AR Path="/5F8FBDC2/5FA1E6B6" Ref="#PE0101"  Part="1"
+F 0 "#PE0101" H 12050 2300 50  0001 C CNN
+F 1 "PE" V 11950 2325 59  0000 R TNN
+F 2 "" H 12050 2300 50  0001 C CNN
+F 3 "" H 12050 2300 50  0001 C CNN
+	1    12050 2300
+	-1   0    0    1
+$EndComp
+$Comp
+L TFT_LCD_Audio_USB-rescue:GND-EEZ_DIB_MCU_r3B4-eagle-import #SUPPLY?
+U 1 1 5FA1FA59
+P 11950 2300
+AR Path="/B3D79DE65FA1FA59" Ref="#SUPPLY?"  Part="1"
+AR Path="/5F88D857/B3D79DE65FA1FA59" Ref="#SUPPLY?"  Part="1"
+AR Path="/5F8FBDC2/5FA1FA59" Ref="#SUPPLY0101"  Part="1"
+F 0 "#SUPPLY0101" H 11950 2300 50  0001 C CNN
+F 1 "GND" H 11850 2150 59  0000 L BNN
+F 2 "" H 11950 2300 50  0001 C CNN
+F 3 "" H 11950 2300 50  0001 C CNN
+	1    11950 2300
+	-1   0    0    1
+$EndComp
+Wire Wire Line
+	11650 2700 11200 2700
+Wire Wire Line
+	11200 2700 11200 2350
+Wire Wire Line
+	11200 2350 10500 2350
+Wire Wire Line
+	10500 2350 10500 2700
+Connection ~ 10500 2700
+Wire Wire Line
+	10500 2700 10600 2700
+Wire Wire Line
+	11650 2800 11150 2800
+Wire Wire Line
+	11150 2800 11150 2400
+Wire Wire Line
+	11150 2400 10550 2400
+Wire Wire Line
+	10550 2400 10550 2800
+Connection ~ 10550 2800
+Wire Wire Line
+	10550 2800 10600 2800
+Wire Wire Line
+	11650 2600 11250 2600
+Wire Wire Line
+	11250 2600 11250 2250
+Wire Wire Line
+	11250 2250 10350 2250
+Wire Wire Line
+	10350 2250 10350 2900
+Connection ~ 10350 2900
+Wire Wire Line
+	10350 2900 10600 2900
+Wire Wire Line
+	10600 2200 11200 2200
+Wire Wire Line
+	11650 3000 11250 3000
+Wire Wire Line
+	11250 3000 11250 3950
+Wire Wire Line
+	11250 3950 9700 3950
+Wire Wire Line
+	9700 3950 9700 2600
+Connection ~ 9700 2600
+Wire Wire Line
+	9700 2600 10200 2600
 $EndSCHEMATC
