File: serdes.sch (KiCad schematic (older format))
At the start: 1 part, among them U1 LFE5U-85F-6BG381C

Commit message: Routing SERDES
Parts:
- added C14, C15, C16, C18, C21, C33, C34, C35, C47, C52: 22nF, Capacitor_SMD:C_0603_1608Metric, symbol Device:C
Connections:
- net S_3_P: now reaches U1.W17 (HDTXP0_D1CH1)
- net S_3_P: now also C21.2
- net S_3_N: now reaches U1.W18 (HDTXN0_D1CH1)
- net S_3_N: now also C52.2
- net S_CLK_P: now reaches U1.Y11 (REFCLKP_D0)
- net S_CLK_P: now also C14.2
- net S_CLK_N: now reaches U1.Y12 (REFCLKN_D0)
- net S_CLK_N: now also C33.2
- net S_2_P: now reaches U1.Y14 (HDRXP0_D1CH0)
- net S_2_P: now also C18.2
- net S_2_N: now reaches U1.Y15 (HDRXN0_D1CH0)
- net S_2_N: now also C47.2
- net S_0_P: now reaches U1.Y5 (HDRXP0_D0CH0)
- net S_0_P: now also C15.2
- net S_0_N: now reaches U1.Y6 (HDRXN0_D0CH0)
- net S_0_N: now also C34.2
- net S_1_P: now reaches U1.Y7 (HDRXP0_D0CH1)
- net S_1_P: now also C16.2
- net S_1_N: now reaches U1.Y8 (HDRXN0_D0CH1)
- net S_1_N: now also C35.2
- new net SRCLKN: C33.1
- new net SRCLKP: C14.1
- new net SRXN00: C34.1
- new net SRXN01: C35.1
- new net SRXN10: C47.1
- new net SRXP00: C15.1
- new net SRXP01: C16.1
- new net SRXP10: C18.1
- new net STXN11: C52.1
- new net STXP11: C21.1
- no-connect marks 8 -> 10
Changed lines of the file:
@@
 NoConn ~ 4850 2050
 NoConn ~ 4850 2250
-NoConn ~ 6550 3500
-NoConn ~ 6550 3700
-NoConn ~ 4850 3700
-NoConn ~ 4850 3500
 Wire Wire Line
 	6550 3150 6650 3150
@@
 Wire Wire Line
 	6650 3200 6650 3250
+NoConn ~ 6550 3400
+NoConn ~ 6550 3500
+NoConn ~ 4850 3400
+NoConn ~ 4850 3500
+$Comp
+L Device:C C?
+U 1 1 5FA1880E
+P 4300 1950
+AR Path="/5FA1880E" Ref="C?"  Part="1"
+AR Path="/58D51CAD/5FA1880E" Ref="C?"  Part="1"
+AR Path="/58DA7327/5FA1880E" Ref="C14"  Part="1"
+F 0 "C14" H 4325 2050 50  0000 L CNN
+F 1 "22nF" V 4350 2100 50  0000 L CNN
+F 2 "Capacitor_SMD:C_0603_1608Metric" H 4338 1800 50  0001 C CNN
+F 3 "" H 4300 1950 50  0000 C CNN
+F 4 "CX0603MRX7R8BB223" H 4300 1950 50  0001 C CNN "MPN"
+	1    4300 1950
+	0    -1   -1   0
+$EndComp
+$Comp
+L Device:C C?
+U 1 1 5FA19032
+P 4300 2150
+AR Path="/5FA19032" Ref="C?"  Part="1"
+AR Path="/58D51CAD/5FA19032" Ref="C?"  Part="1"
+AR Path="/58DA7327/5FA19032" Ref="C15"  Part="1"
+F 0 "C15" H 4325 2250 50  0000 L CNN
+F 1 "22nF" V 4350 2300 50  0000 L CNN
+F 2 "Capacitor_SMD:C_0603_1608Metric" H 4338 2000 50  0001 C CNN
+F 3 "" H 4300 2150 50  0000 C CNN
+F 4 "CX0603MRX7R8BB223" H 4300 2150 50  0001 C CNN "MPN"
+	1    4300 2150
+	0    -1   -1   0
+$EndComp
+$Comp
+L Device:C C?
+U 1 1 5FA1953D
+P 4300 2350
+AR Path="/5FA1953D" Ref="C?"  Part="1"
+AR Path="/58D51CAD/5FA1953D" Ref="C?"  Part="1"
+AR Path="/58DA7327/5FA1953D" Ref="C16"  Part="1"
+F 0 "C16" H 4325 2450 50  0000 L CNN
+F 1 "22nF" V 4350 2500 50  0000 L CNN
+F 2 "Capacitor_SMD:C_0603_1608Metric" H 4338 2200 50  0001 C CNN
+F 3 "" H 4300 2350 50  0000 C CNN
+F 4 "CX0603MRX7R8BB223" H 4300 2350 50  0001 C CNN "MPN"
+	1    4300 2350
+	0    -1   -1   0
+$EndComp
+$Comp
+L Device:C C?
+U 1 1 5FA2060C
+P 7000 1950
+AR Path="/5FA2060C" Ref="C?"  Part="1"
+AR Path="/58D51CAD/5FA2060C" Ref="C?"  Part="1"
+AR Path="/58DA7327/5FA2060C" Ref="C33"  Part="1"
+F 0 "C33" H 7025 2050 50  0000 L CNN
+F 1 "22nF" V 7050 2100 50  0000 L CNN
+F 2 "Capacitor_SMD:C_0603_1608Metric" H 7038 1800 50  0001 C CNN
+F 3 "" H 7000 1950 50  0000 C CNN
+F 4 "CX0603MRX7R8BB223" H 7000 1950 50  0001 C CNN "MPN"
+	1    7000 1950
+	0    1    1    0
+$EndComp
+$Comp
+L Device:C C?
+U 1 1 5FA20D19
+P 7000 2150
+AR Path="/5FA20D19" Ref="C?"  Part="1"
+AR Path="/58D51CAD/5FA20D19" Ref="C?"  Part="1"
+AR Path="/58DA7327/5FA20D19" Ref="C34"  Part="1"
+F 0 "C34" H 7025 2250 50  0000 L CNN
+F 1 "22nF" V 7050 2300 50  0000 L CNN
+F 2 "Capacitor_SMD:C_0603_1608Metric" H 7038 2000 50  0001 C CNN
+F 3 "" H 7000 2150 50  0000 C CNN
+F 4 "CX0603MRX7R8BB223" H 7000 2150 50  0001 C CNN "MPN"
+	1    7000 2150
+	0    1    1    0
+$EndComp
+$Comp
+L Device:C C?
+U 1 1 5FA214AC
+P 7000 2350
+AR Path="/5FA214AC" Ref="C?"  Part="1"
+AR Path="/58D51CAD/5FA214AC" Ref="C?"  Part="1"
+AR Path="/58DA7327/5FA214AC" Ref="C35"  Part="1"
+F 0 "C35" H 7025 2450 50  0000 L CNN
+F 1 "22nF" V 7050 2500 50  0000 L CNN
+F 2 "Capacitor_SMD:C_0603_1608Metric" H 7038 2200 50  0001 C CNN
+F 3 "" H 7000 2350 50  0000 C CNN
+F 4 "CX0603MRX7R8BB223" H 7000 2350 50  0001 C CNN "MPN"
+	1    7000 2350
+	0    1    1    0
+$EndComp
+$Comp
+L Device:C C?
+U 1 1 5FA36FAD
+P 4300 3600
+AR Path="/5FA36FAD" Ref="C?"  Part="1"
+AR Path="/58D51CAD/5FA36FAD" Ref="C?"  Part="1"
+AR Path="/58DA7327/5FA36FAD" Ref="C18"  Part="1"
+F 0 "C18" H 4325 3700 50  0000 L CNN
+F 1 "22nF" V 4450 3550 50  0000 L CNN
+F 2 "Capacitor_SMD:C_0603_1608Metric" H 4338 3450 50  0001 C CNN
+F 3 "" H 4300 3600 50  0000 C CNN
+F 4 "CX0603MRX7R8BB223" H 4300 3600 50  0001 C CNN "MPN"
+	1    4300 3600
+	0    -1   -1   0
+$EndComp
+$Comp
+L Device:C C?
+U 1 1 5FA377C2
+P 4300 3700
+AR Path="/5FA377C2" Ref="C?"  Part="1"
+AR Path="/58D51CAD/5FA377C2" Ref="C?"  Part="1"
+AR Path="/58DA7327/5FA377C2" Ref="C21"  Part="1"
+F 0 "C21" H 4325 3800 50  0000 L CNN
+F 1 "22nF" V 4150 3650 50  0000 L CNN
+F 2 "Capacitor_SMD:C_0603_1608Metric" H 4338 3550 50  0001 C CNN
+F 3 "" H 4300 3700 50  0000 C CNN
+F 4 "CX0603MRX7R8BB223" H 4300 3700 50  0001 C CNN "MPN"
+	1    4300 3700
+	0    -1   -1   0
+$EndComp
+NoConn ~ 6550 3800
+NoConn ~ 4850 3800
+$Comp
+L Device:C C?
+U 1 1 5FA4BE8F
+P 7000 3600
+AR Path="/5FA4BE8F" Ref="C?"  Part="1"
+AR Path="/58D51CAD/5FA4BE8F" Ref="C?"  Part="1"
+AR Path="/58DA7327/5FA4BE8F" Ref="C47"  Part="1"
+F 0 "C47" H 7025 3700 50  0000 L CNN
+F 1 "22nF" V 6850 3550 50  0000 L CNN
+F 2 "Capacitor_SMD:C_0603_1608Metric" H 7038 3450 50  0001 C CNN
+F 3 "" H 7000 3600 50  0000 C CNN
+F 4 "CX0603MRX7R8BB223" H 7000 3600 50  0001 C CNN "MPN"
+	1    7000 3600
+	0    1    1    0
+$EndComp
+$Comp
+L Device:C C?
+U 1 1 5FA4C4EC
+P 7000 3700
+AR Path="/5FA4C4EC" Ref="C?"  Part="1"
+AR Path="/58D51CAD/5FA4C4EC" Ref="C?"  Part="1"
+AR Path="/58DA7327/5FA4C4EC" Ref="C52"  Part="1"
+F 0 "C52" H 7025 3800 50  0000 L CNN
+F 1 "22nF" V 7150 3650 50  0000 L CNN
+F 2 "Capacitor_SMD:C_0603_1608Metric" H 7038 3550 50  0001 C CNN
+F 3 "" H 7000 3700 50  0000 C CNN
+F 4 "CX0603MRX7R8BB223" H 7000 3700 50  0001 C CNN "MPN"
+	1    7000 3700
+	0    1    1    0
+$EndComp
+Text GLabel 4150 1950 0    60   Input ~ 0
+SRCLKP
+Text GLabel 4150 2150 0    60   Input ~ 0
+SRXP00
+Text GLabel 4150 2350 0    60   Input ~ 0
+SRXP01
+Text GLabel 4150 3600 0    60   Input ~ 0
+SRXP10
+Text GLabel 4150 3700 0    60   Input ~ 0
+STXP11
+Text GLabel 7150 1950 2    60   Input ~ 0
+SRCLKN
+Text GLabel 7150 2350 2    60   Input ~ 0
+SRXN01
+Text GLabel 7150 3600 2    60   Input ~ 0
+SRXN10
+Text GLabel 7150 3700 2    60   Input ~ 0
+STXN11
+Text GLabel 7150 2150 2    60   Input ~ 0
+SRXN00
+Wire Wire Line
+	4450 1950 4850 1950
+Wire Wire Line
+	4850 2150 4450 2150
+Wire Wire Line
+	4450 2350 4850 2350
+Wire Wire Line
+	6550 1950 6850 1950
+Wire Wire Line
+	6850 2150 6550 2150
+Wire Wire Line
+	6850 2350 6550 2350
+Wire Wire Line
+	6550 3600 6850 3600
+Wire Wire Line
+	6850 3700 6550 3700
+Wire Wire Line
+	4450 3600 4850 3600
+Wire Wire Line
+	4450 3700 4850 3700
+Text Label 4500 1950 0    60   ~ 0
+S_CLK_P
+Text Label 4500 2150 0    60   ~ 0
+S_0_P
+Text Label 4500 2350 0    60   ~ 0
+S_1_P
+Text Label 4450 3600 0    60   ~ 0
+S_2_P
+Text Label 4450 3700 0    60   ~ 0
+S_3_P
+Text Label 6600 1950 0    60   ~ 0
+S_CLK_N
+Text Label 6650 2150 0    60   ~ 0
+S_0_N
+Text Label 6650 2350 0    60   ~ 0
+S_1_N
+Text Label 6650 3600 0    60   ~ 0
+S_2_N
+Text Label 6650 3700 0    60   ~ 0
+S_3_N
 $EndSCHEMATC
