File: ulx3s.sch (KiCad schematic (older format))
At the start: 4 parts

Commit message: Rewiering LCD OUT to bottom left
Parts:
- H1, H2, H3, H4: footprint Mounting_Holes:MountingHole_3.2mm_M3_ISO14580_Pad -> MountingHole:MountingHole_3.2mm_M3_ISO14580_Pad
Changed lines of the file:
@@
 F 0 "H1" H 3150 6450 50  0000 C CNN
 F 1 "HOLE" V 3250 6350 50  0000 C CNN
-F 2 "Mounting_Holes:MountingHole_3.2mm_M3_ISO14580_Pad" H 3150 6350 50  0001 C CNN
+F 2 "MountingHole:MountingHole_3.2mm_M3_ISO14580_Pad" H 3150 6350 50  0001 C CNN
 F 3 "" H 3150 6350 50  0000 C CNN
 	1    3150 6350
@@
 F 0 "H2" H 4250 6450 50  0000 C CNN
 F 1 "HOLE" V 4350 6350 50  0000 C CNN
-F 2 "Mounting_Holes:MountingHole_3.2mm_M3_ISO14580_Pad" H 4250 6350 50  0001 C CNN
+F 2 "MountingHole:MountingHole_3.2mm_M3_ISO14580_Pad" H 4250 6350 50  0001 C CNN
 F 3 "" H 4250 6350 50  0000 C CNN
 	1    4250 6350
@@
 F 0 "H3" H 4250 5750 50  0000 C CNN
 F 1 "HOLE" V 4350 5650 50  0000 C CNN
-F 2 "Mounting_Holes:MountingHole_3.2mm_M3_ISO14580_Pad" H 4250 5650 50  0001 C CNN
+F 2 "MountingHole:MountingHole_3.2mm_M3_ISO14580_Pad" H 4250 5650 50  0001 C CNN
 F 3 "" H 4250 5650 50  0000 C CNN
 	1    4250 5650
@@
 F 0 "H4" H 3150 5750 50  0000 C CNN
 F 1 "HOLE" V 3250 5650 50  0000 C CNN
-F 2 "Mounting_Holes:MountingHole_3.2mm_M3_ISO14580_Pad" H 3150 5650 50  0001 C CNN
+F 2 "MountingHole:MountingHole_3.2mm_M3_ISO14580_Pad" H 3150 5650 50  0001 C CNN
 F 3 "" H 3150 5650 50  0000 C CNN
 F 4 "Leave empty" H 3150 5650 50  0001 C CNN "Note"
